Commit message: Added "${prefix}" variable so that multiple instances of the EZGripper can be instantiated in a robot URDF and each will have a unique name defined by "${prefix}" value.

File: ezgripper_driver/urdf/ezgripper_quad.urdf.xacro (robot description, xacro)
@@ -1,8 +1,7 @@
 <?xml version="1.0" encoding="UTF-8"?>
 <robot name="ezgripper" xmlns:xacro="http://www.ros.org/wiki/xacro">
-<!--macro name="ezgripper" params="*origin"-->
-<macro name="ezgripper_quad" params="parent_link *origin">
+<macro name="ezgripper_quad" params="prefix parent_link *origin">
     <!-- links -->
-    <link name="palm_link">
+    <link name="${prefix}_ezgripper_palm_link">
       <visual>
         <origin xyz="0 0 0" rpy="0 0 0"/>
@@ -22,14 +21,27 @@
     </inertial>
     </link>
-    <joint name="ezgripper_connect" type="fixed">
+    <joint name="${prefix}_ezgripper_connect" type="fixed">
         <origin rpy="-1.57 0 0" xyz="0.049 0.0 0.2"/>
         <parent link="${parent_link}"/>
-        <child link="palm_link"/>
+        <child link="${prefix}_ezgripper_palm_link"/>
         <axis xyz="0 0 0"/>
         <limit effort="0" lower="-1.57075" upper="0.25" velocity="3.67"/>
     </joint>
+    <ezgripper_finger prefix="${prefix}" postfix="1" reflect="1"/>
+    <ezgripper_finger prefix="${prefix}" postfix="2" reflect="1"/>
+    <ezgripper_finger prefix="${prefix}" postfix="3" reflect="1"/>
+    <ezgripper_finger prefix="${prefix}" postfix="4" reflect="1"/>
+    <ezgripper_knuckle prefix="${prefix}" postfix="1" reflectY="1" reflectZ="1" reflectR="1" mimic_test="false"/>
+    <ezgripper_knuckle prefix="${prefix}" postfix="2" reflectY="-1" reflectZ="1" reflectR="-1" mimic_test="true"/>
+    <ezgripper_knuckle prefix="${prefix}" postfix="3" reflectY="1" reflectZ="-1" reflectR="1" mimic_test="true"/>
+    <ezgripper_knuckle prefix="${prefix}" postfix="4" reflectY="-1" reflectZ="-1" reflectR="-1" mimic_test="true"/>
+    <ezgripper_knuckle_trans prefix="${prefix}" postfix="1"/>
+    <ezgripper_knuckle_trans prefix="${prefix}" postfix="2"/>
+    <ezgripper_knuckle_trans prefix="${prefix}" postfix="3"/>
+    <ezgripper_knuckle_trans prefix="${prefix}" postfix="4"/>
+    <gazebo_knuckle_jsp prefix="${prefix}" />
 </macro>
-<macro name="finger" params="postfix reflect">
-    <link name="finger_${postfix}">
+<macro name="ezgripper_finger" params="prefix postfix reflect">
+    <link name="${prefix}_ezgripper_finger_${postfix}">
       <visual>
         <origin xyz="0 0 0" rpy="0 0 0"/>
@@ -50,33 +62,25 @@
     </link>
 </macro>
-<finger postfix="1" reflect="1"/>
-<finger postfix="2" reflect="1"/>
-<finger postfix="3" reflect="1"/>
-<finger postfix="4" reflect="1"/>
     <!-- joints -->
-<macro name="knuckle" params="postfix reflectY reflectZ reflectR mimic_test">
-    <joint name="knuckle_${postfix}" type="revolute">
-      <parent link="palm_link"/>
-      <child link="finger_${postfix}"/>
+<macro name="ezgripper_knuckle" params="prefix postfix reflectY reflectZ reflectR mimic_test">
+    <joint name="${prefix}_ezgripper_knuckle_${postfix}" type="revolute">
+      <parent link="${prefix}_ezgripper_palm_link"/>
+      <child link="${prefix}_ezgripper_finger_${postfix}"/>
       <origin xyz="0.1056 ${reflectY*0.03} ${reflectZ*0.03}" rpy="${1.5708 * reflectR} 0 3.14159"/>
       <axis xyz="0 1 0"/>
       <limit lower="-.27" upper="1.57075" effort="1" velocity="3.67"/>
       <xacro:if value="${mimic_test}">
-           <mimic joint="knuckle_1"/>
+           <mimic joint="${prefix}_ezgripper_knuckle_1"/>
       </xacro:if>
     </joint>
 </macro>
-<knuckle postfix="1" reflectY="1" reflectZ="1" reflectR="1" mimic_test="false"/>
-<knuckle postfix="2" reflectY="-1" reflectZ="1" reflectR="-1" mimic_test="true"/>
-<knuckle postfix="3" reflectY="1" reflectZ="-1" reflectR="1" mimic_test="true"/>
-<knuckle postfix="4" reflectY="-1" reflectZ="-1" reflectR="-1" mimic_test="true"/>
     <!-- transmissions for Gazebo -->
-<macro name="knuckle_trans" params="postfix">
-   <transmission name="ezgripper_trans_${postfix}">
+<macro name="ezgripper_knuckle_trans" params="prefix postfix">
+   <transmission name="${prefix}_ezgripper_trans_${postfix}">
       <type>transmission_interface/SimpleTransmission</type>
-      <joint name="knuckle_${postfix}">
+      <joint name="${prefix}_ezgripper_knuckle_${postfix}">
          <hardwareInterface>PositionJointInterface</hardwareInterface>
       </joint>
-      <actuator name="ezgripper_motor${postfix}">
+      <actuator name="${prefix}_ezgripper_motor${postfix}">
          <mechanicalReduction>1</mechanicalReduction>
          <hardwareInterface>PositionJointInterface</hardwareInterface>
@@ -84,13 +88,11 @@
    </transmission>
 </macro>
-<knuckle_trans postfix="1"/>
-<knuckle_trans postfix="2"/>
-<knuckle_trans postfix="3"/>
-<knuckle_trans postfix="4"/>
-<gazebo>
-  <plugin name="joint_state_publisher" filename="libgazebo_ros_joint_state_publisher.so">
-    <jointName>knuckle_1,knuckle_2,knuckle_3,knuckle_4  </jointName>
-  </plugin>
-</gazebo>
+<macro name="gazebo_knuckle_jsp" params="prefix">
+    <gazebo>
+      <plugin name="joint_state_publisher" filename="libgazebo_ros_joint_state_publisher.so">
+        <jointName>${prefix}_ezgripper_knuckle_1,${prefix}_ezgripper_knuckle_2,${prefix}_ezgripper_knuckle_3,${prefix}_ezgripper_knuckle_4  </jointName>
+      </plugin>
+    </gazebo>
+</macro>
 <gazebo>
    <plugin name="gazebo_ros_control" filename="libgazebo_ros_control.so">
