Commit message: Changes for urdf to support Gazebo

File: ezgripper_driver/urdf/ezgripper_dual.urdf.xacro (robot description, xacro)
@@ -1,6 +1,6 @@
-<?xml version="1.0"?>
+<?xml version="1.0" encoding="UTF-8"?>
 <robot name="ezgripper" xmlns:xacro="http://www.ros.org/wiki/xacro">
 <!--macro name="ezgripper" params="*origin"-->
-<macro name="ezgripper" params="parent_link *origin">
+<macro name="ezgripper_dual" params="parent_link *origin">
     <!-- links -->
     <link name="palm_link">
@@ -19,17 +19,17 @@
     <inertial>
       <mass value=".3"/>
-      <inertia ixx="0.03" ixy="0.0" ixz="0.0" iyy="1.0" iyz="0.0" izz="0.0"/>
+      <inertia ixx="0.01" ixy="0.0" ixz="0.0" iyy="0.01" iyz="0.0" izz="0.01"/>
     </inertial>
     </link>
     <joint name="ezgripper_connect" type="fixed">
-        <xacro:insert_block name="origin"/>
+        <origin rpy="-1.57 0 0" xyz="0.049 0.0 0.2"/>
         <parent link="${parent_link}"/>
         <child link="palm_link"/>
-      <axis xyz="0 0 0"/>
-      <limit lower="-1.57075" upper="0.25" effort="0" velocity="3.67"/>
+        <axis xyz="0 0 0"/>
+        <limit effort="0" lower="-1.57075" upper="0.25" velocity="3.67"/>
     </joint>
 </macro>
 <macro name="finger" params="postfix reflect">
-    <link name="finger_${postfix}">j
+    <link name="finger_${postfix}">
       <visual>
         <origin xyz="0 0 0" rpy="0 0 0"/>
@@ -44,22 +44,20 @@
         </geometry>
       </collision>
-    <inertial>
-      <mass value=".025"/>
-      <inertia ixx="0.062" ixy="0.0" ixz="0.0" iyy="1.0" iyz="0.0" izz="0.0"/>
-    </inertial>
-     </link>
+      <inertial>
+        <mass value=".025"/>
+        <inertia ixx="0.01" ixy="0.0" ixz="0.0" iyy="0.01" iyz="0.0" izz="0.01"/>
+      </inertial>
+    </link>
 </macro>
 <finger postfix="1" reflect="1" />
 <finger postfix="2" reflect="1" />
-<finger postfix="3" reflect="1" />
-<finger postfix="4" reflect="1" />
     <!-- joints -->
-<macro name="knuckle" params="postfix reflectY reflectZ mimic_test">
+<macro name="knuckle" params="postfix reflectY reflectZ reflectR mimic_test">
     <joint name="knuckle_${postfix}" type="revolute">
       <parent link="palm_link"/>
       <child link="finger_${postfix}"/>
-      <origin xyz="0.088 ${reflectY*0.025} ${reflectZ*0.025}" rpy="${(0.5-0.5*reflectZ)*3.14159} 0 0"/>
+      <origin xyz="0.1056 ${reflectY*0.03} 0" rpy="${1.5708 * reflectR} 0 3.14159"/>
       <axis xyz="0 1 0"/>
-      <limit lower="-1.57075" upper="0.25" effort="0" velocity="3.67"/>
+      <limit lower="-.27" upper="1.57075" effort="1" velocity="3.67"/>
       <xacro:if value="${mimic_test}">
            <mimic joint="knuckle_1"/>
@@ -67,17 +65,29 @@
     </joint>
 </macro>
-<knuckle postfix="1" reflectY="1" reflectZ="1" mimic_test="false"/>
-<knuckle postfix="2" reflectY="-1" reflectZ="1" mimic_test="true"/>
-<knuckle postfix="3" reflectY="1" reflectZ="-1" mimic_test="true"/>
-<knuckle postfix="4" reflectY="-1" reflectZ="-1" mimic_test="true"/>
-<macro name="gazebostuff" params="postfix2">
-  <gazebo reference="knuckle_${postfix2}">
-    <provideFeedback>1</provideFeedback>
-    <implicitSpringDamper>1</implicitSpringDamper>
-  </gazebo>
+<knuckle postfix="1" reflectY="1" reflectZ="1" reflectR="1" mimic_test="false"/>
+<knuckle postfix="2" reflectY="-1" reflectZ="1" reflectR="-1" mimic_test="true"/>
+    <!-- transmissions for Gazebo -->
+<macro name="knuckle_trans" params="postfix">
+   <transmission name="ezgripper_trans_${postfix}">
+      <type>transmission_interface/SimpleTransmission</type>
+      <joint name="knuckle_${postfix}">
+         <hardwareInterface>PositionJointInterface</hardwareInterface>
+      </joint>
+      <actuator name="ezgripper_motor${postfix}">
+         <mechanicalReduction>1</mechanicalReduction>
+         <hardwareInterface>PositionJointInterface</hardwareInterface>
+      </actuator>
+   </transmission>
 </macro>
-<gazebostuff postfix2="1"/>
-<gazebostuff postfix2="2"/>
-<gazebostuff postfix2="3"/>
-<gazebostuff postfix2="4"/>
+<knuckle_trans postfix="1"/>
+<knuckle_trans postfix="2"/>
+<gazebo>
+  <plugin name="joint_state_publisher" filename="libgazebo_ros_joint_state_publisher.so">
+    <jointName>knuckle_1,knuckle_2  </jointName>
+  </plugin>
+</gazebo>
+<gazebo>
+   <plugin name="gazebo_ros_control" filename="libgazebo_ros_control.so">
+   </plugin>
+</gazebo>
 </robot>

File: ezgripper_driver/urdf/ezgripper_quad.urdf.xacro (robot description, xacro)
@@ -1,3 +1,3 @@
-<?xml version="1.0"?>
+<?xml version="1.0" encoding="UTF-8"?>
 <robot name="ezgripper" xmlns:xacro="http://www.ros.org/wiki/xacro">
 <!--macro name="ezgripper" params="*origin"-->
@@ -19,13 +19,13 @@
     <inertial>
       <mass value=".3"/>
-      <inertia ixx="0.03" ixy="0.0" ixz="0.0" iyy="1.0" iyz="0.0" izz="0.0"/>
+      <inertia ixx="0.01" ixy="0.0" ixz="0.0" iyy="0.01" iyz="0.0" izz="0.01"/>
     </inertial>
     </link>
     <joint name="ezgripper_connect" type="fixed">
-        <xacro:insert_block name="origin"/>
+        <origin rpy="-1.57 0 0" xyz="0.049 0.0 0.2"/>
         <parent link="${parent_link}"/>
         <child link="palm_link"/>
-      <axis xyz="0 0 0"/>
-      <limit lower="-1.57075" upper="0.25" effort="0" velocity="3.67"/>
+        <axis xyz="0 0 0"/>
+        <limit effort="0" lower="-1.57075" upper="0.25" velocity="3.67"/>
     </joint>
 </macro>
@@ -44,14 +44,14 @@
         </geometry>
       </collision>
-    <inertial>
-      <mass value=".025"/>
-      <inertia ixx="0.062" ixy="0.0" ixz="0.0" iyy="1.0" iyz="0.0" izz="0.0"/>
-    </inertial>
-     </link>
+      <inertial>
+        <mass value=".025"/>
+        <inertia ixx="0.01" ixy="0.0" ixz="0.0" iyy=".01" iyz="0.0" izz="0.01"/>
+      </inertial>
+    </link>
 </macro>
-<finger postfix="1" reflect="1" />
-<finger postfix="2" reflect="1" />
-<finger postfix="3" reflect="1" />
-<finger postfix="4" reflect="1" />
+<finger postfix="1" reflect="1"/>
+<finger postfix="2" reflect="1"/>
+<finger postfix="3" reflect="1"/>
+<finger postfix="4" reflect="1"/>
     <!-- joints -->
 <macro name="knuckle" params="postfix reflectY reflectZ reflectR mimic_test">
@@ -59,7 +59,7 @@
       <parent link="palm_link"/>
       <child link="finger_${postfix}"/>
-      <origin xyz="0.1056 ${reflectY*0.03} ${reflectZ*0.03}" rpy="${1.5708 * reflectR} 0 0"/>
+      <origin xyz="0.1056 ${reflectY*0.03} ${reflectZ*0.03}" rpy="${1.5708 * reflectR} 0 3.14159"/>
       <axis xyz="0 1 0"/>
-      <limit lower="-1.57075" upper="-3.42" effort="0" velocity="3.67"/>
+      <limit lower="-.27" upper="1.57075" effort="1" velocity="3.67"/>
       <xacro:if value="${mimic_test}">
            <mimic joint="knuckle_1"/>
@@ -71,13 +71,29 @@
 <knuckle postfix="3" reflectY="1" reflectZ="-1" reflectR="1" mimic_test="true"/>
 <knuckle postfix="4" reflectY="-1" reflectZ="-1" reflectR="-1" mimic_test="true"/>
-<macro name="gazebostuff" params="postfix2">
-  <gazebo reference="knuckle_${postfix2}">
-    <provideFeedback>1</provideFeedback>
-    <implicitSpringDamper>1</implicitSpringDamper>
-  </gazebo>
+    <!-- transmissions for Gazebo -->
+<macro name="knuckle_trans" params="postfix">
+   <transmission name="ezgripper_trans_${postfix}">
+      <type>transmission_interface/SimpleTransmission</type>
+      <joint name="knuckle_${postfix}">
+         <hardwareInterface>PositionJointInterface</hardwareInterface>
+      </joint>
+      <actuator name="ezgripper_motor${postfix}">
+         <mechanicalReduction>1</mechanicalReduction>
+         <hardwareInterface>PositionJointInterface</hardwareInterface>
+      </actuator>
+   </transmission>
 </macro>
-<gazebostuff postfix2="1"/>
-<gazebostuff postfix2="2"/>
-<gazebostuff postfix2="3"/>
-<gazebostuff postfix2="4"/>
+<knuckle_trans postfix="1"/>
+<knuckle_trans postfix="2"/>
+<knuckle_trans postfix="3"/>
+<knuckle_trans postfix="4"/>
+<gazebo>
+  <plugin name="joint_state_publisher" filename="libgazebo_ros_joint_state_publisher.so">
+    <jointName>knuckle_1,knuckle_2,knuckle_3,knuckle_4  </jointName>
+  </plugin>
+</gazebo>
+<gazebo>
+   <plugin name="gazebo_ros_control" filename="libgazebo_ros_control.so">
+   </plugin>
+</gazebo>
 </robot>

Commit message: Added ${prefix} variable so that multiple instances of EZGripper can be placed in a robot URDF and each will have a unique identifier defined by ${prefix}.

File: ezgripper_driver/urdf/ezgripper_dual.urdf.xacro (robot description, xacro)
@@ -2,7 +2,7 @@
 <robot name="ezgripper" xmlns:xacro="http://www.ros.org/wiki/xacro">
 <!--macro name="ezgripper" params="*origin"-->
-<macro name="ezgripper_dual" params="parent_link *origin">
+<macro name="ezgripper_dual" params="prefix parent_link *origin">
     <!-- links -->
-    <link name="palm_link">
+    <link name="${prefix}_ezgripper_palm_link">
       <visual>
         <origin xyz="0 0 0" rpy="0 0 0"/>
@@ -22,14 +22,21 @@
     </inertial>
     </link>
-    <joint name="ezgripper_connect" type="fixed">
+    <joint name="${prefix}_ezgripper_connect" type="fixed">
         <origin rpy="-1.57 0 0" xyz="0.049 0.0 0.2"/>
         <parent link="${parent_link}"/>
-        <child link="palm_link"/>
+        <child link="${prefix}_ezgripper_palm_link"/>
         <axis xyz="0 0 0"/>
         <limit effort="0" lower="-1.57075" upper="0.25" velocity="3.67"/>
     </joint>
+    <ezgripper_finger prefix="${prefix}" postfix="1" reflect="1" />
+    <ezgripper_finger prefix="${prefix}" postfix="2" reflect="1" />
+    <ezgripper_knuckle prefix="${prefix}" postfix="1" reflectY="1" reflectZ="1" reflectR="1" mimic_test="false"/>
+    <ezgripper_knuckle prefix="${prefix}" postfix="2" reflectY="-1" reflectZ="1" reflectR="-1" mimic_test="true"/>
+    <ezgripper_knuckle_trans prefix="${prefix}" postfix="1"/>
+    <ezgripper_knuckle_trans prefix="${prefix}" postfix="2"/>
+    <gazebo_knuckle_jsp prefix="${prefix}" />
 </macro>
-<macro name="finger" params="postfix reflect">
-    <link name="finger_${postfix}">
+<macro name="ezgripper_finger" params="prefix postfix reflect">
+    <link name="${prefix}_ezgripper_finger_${postfix}">
       <visual>
         <origin xyz="0 0 0" rpy="0 0 0"/>
@@ -50,29 +57,25 @@
     </link>
 </macro>
-<finger postfix="1" reflect="1" />
-<finger postfix="2" reflect="1" />
     <!-- joints -->
-<macro name="knuckle" params="postfix reflectY reflectZ reflectR mimic_test">
-    <joint name="knuckle_${postfix}" type="revolute">
-      <parent link="palm_link"/>
-      <child link="finger_${postfix}"/>
+<macro name="ezgripper_knuckle" params="prefix postfix reflectY reflectZ reflectR mimic_test">
+    <joint name="${prefix}_ezgripper_knuckle_${postfix}" type="revolute">
+      <parent link="${prefix}_ezgripper_palm_link"/>
+      <child link="${prefix}_ezgripper_finger_${postfix}"/>
       <origin xyz="0.1056 ${reflectY*0.03} 0" rpy="${1.5708 * reflectR} 0 3.14159"/>
       <axis xyz="0 1 0"/>
       <limit lower="-.27" upper="1.57075" effort="1" velocity="3.67"/>
       <xacro:if value="${mimic_test}">
-           <mimic joint="knuckle_1"/>
+           <mimic joint="ezgripper_knuckle_1"/>
       </xacro:if>
     </joint>
 </macro>
-<knuckle postfix="1" reflectY="1" reflectZ="1" reflectR="1" mimic_test="false"/>
-<knuckle postfix="2" reflectY="-1" reflectZ="1" reflectR="-1" mimic_test="true"/>
     <!-- transmissions for Gazebo -->
-<macro name="knuckle_trans" params="postfix">
-   <transmission name="ezgripper_trans_${postfix}">
+<macro name="ezgripper_knuckle_trans" params="prefix postfix">
+   <transmission name="${prefix}_ezgripper_trans_${postfix}">
       <type>transmission_interface/SimpleTransmission</type>
-      <joint name="knuckle_${postfix}">
+      <joint name="${prefix}_ezgripper_knuckle_${postfix}">
          <hardwareInterface>PositionJointInterface</hardwareInterface>
       </joint>
-      <actuator name="ezgripper_motor${postfix}">
+      <actuator name="${prefix}_ezgripper_motor${postfix}">
          <mechanicalReduction>1</mechanicalReduction>
          <hardwareInterface>PositionJointInterface</hardwareInterface>
@@ -80,11 +83,11 @@
    </transmission>
 </macro>
-<knuckle_trans postfix="1"/>
-<knuckle_trans postfix="2"/>
-<gazebo>
-  <plugin name="joint_state_publisher" filename="libgazebo_ros_joint_state_publisher.so">
-    <jointName>knuckle_1,knuckle_2  </jointName>
-  </plugin>
-</gazebo>
+<macro name="gazeobo_knuckle_jsp" params="prefix">
+   <gazebo>
+     <plugin name="joint_state_publisher" filename="libgazebo_ros_joint_state_publisher.so">
+       <jointName>${prefix}_ezgripper_knuckle_1,${prefix}_ezgripper_knuckle_2  </jointName>
+     </plugin>
+   </gazebo>
+</macro>
 <gazebo>
    <plugin name="gazebo_ros_control" filename="libgazebo_ros_control.so">
