Commit message: Update and rename ezgripper_dual.urdf.xacro to ezgripper_dual_gen2.urdf.xacro
URDF for EZGripper Gen2 Dual robotic gripper.  This is the simple model with no under-actuation.  L1 and L2 are in extended position.

File: ezgripper_driver/urdf/ezgripper_dual_gen2.urdf.xacro (robot description, xacro)
@@ -2,5 +2,5 @@
 <robot name="ezgripper" xmlns:xacro="http://www.ros.org/wiki/xacro">
 <!--macro name="ezgripper" params="*origin"-->
-<macro name="ezgripper_dual" params="prefix parent_link *origin">
+<macro name="ezgripper_dual_gen2" params="prefix parent_link *origin">
     <!-- links -->
     <link name="${prefix}_ezgripper_palm_link">
@@ -8,5 +8,5 @@
         <origin xyz="0 0 0" rpy="0 0 0"/>
         <geometry>
-          <mesh filename="package://ezgripper_driver/meshes/visual/SAKE_Palm_Dual.stl"/>
+          <mesh filename="package://ezgripper_driver/meshes/visual/SAKE_Palm_Dual_Gen2.stl"/>
         </geometry>
       </visual>
@@ -14,5 +14,5 @@
         <origin xyz="0 0 0" rpy="0 0 0"/>
         <geometry>
-          <mesh filename="package://ezgripper_driver/meshes/collision/SAKE_Palm_Dual.stl"/>
+          <mesh filename="package://ezgripper_driver/meshes/collision/SAKE_Palm_Dual_Gen2.stl"/>
         </geometry>
       </collision>
@@ -42,5 +42,5 @@
         <origin xyz="0 0 0" rpy="0 0 0"/>
         <geometry>
-          <mesh filename="package://ezgripper_driver/meshes/visual/SAKE_Finger.stl"/>
+          <mesh filename="package://ezgripper_driver/meshes/visual/SAKE_Finger_Gen2.stl"/>
         </geometry>
       </visual>
@@ -48,5 +48,5 @@
         <origin xyz="0 0 0" rpy="0 0 0"/>
         <geometry>
-          <mesh filename="package://ezgripper_driver/meshes/collision/SAKE_Finger.stl"/>
+          <mesh filename="package://ezgripper_driver/meshes/collision/SAKE_Finger_Gen2.stl"/>
         </geometry>
       </collision>
