Commit message: Fixed passing origin into ezgripper_dual_articulated.urdf.xacro

File: ezgripper_driver/urdf/ezgripper_dual_gen2_articulated.urdf.xacro (robot description, xacro)
@@ -23,5 +23,6 @@
     </link>
     <joint name="${prefix}_ezgripper_connect" type="fixed">
-        <origin rpy="0 0 0" xyz="0.049 0.0 0.2"/>
+        <xacro:insert_block name="origin" />
+        <!-- <origin rpy="0 0 0" xyz="0.049 0.0 0.2"/> -->
         <parent link="${parent_link}"/>
         <child link="${prefix}_ezgripper_palm_link"/>

Commit message: fix xacro namespaces

File: ezgripper_driver/urdf/ezgripper_dual_gen2_articulated.urdf.xacro (robot description, xacro)
@@ -1,6 +1,6 @@
 <?xml version="1.0" encoding="UTF-8"?>
-<robot name="ezgripper" xmlns:xacro="http://www.ros.org/wiki/xacro">
-<!--macro name="ezgripper" params="*origin"-->
-<macro name="ezgripper_dual" params="prefix parent_link *origin">
+<robot name="ezgripper" xmlns:xacro="http://ros.org/wiki/xacro">
+<!--xacro:macro name="ezgripper" params="*origin"-->
+<xacro:macro name="ezgripper_dual" params="prefix parent_link *origin">
     <!-- links -->
     <link name="${prefix}_ezgripper_palm_link">
@@ -40,6 +40,6 @@
     <ezgripper_knuckle_trans prefix="${prefix}" postfix="L1_L2_1"/>
     <gazebo_knuckle_jsp prefix="${prefix}" />
-</macro>
-<macro name="ezgripper_finger_L1" params="prefix postfix reflect">
+</xacro:macro>
+<xacro:macro name="ezgripper_finger_L1" params="prefix postfix reflect">
     <link name="${prefix}_ezgripper_finger_L1_${postfix}">
       <visual>
@@ -60,6 +60,6 @@
       </inertial>
     </link>
-</macro>
-<macro name="ezgripper_finger_L2" params="prefix postfix reflect">
+</xacro:macro>
+<xacro:macro name="ezgripper_finger_L2" params="prefix postfix reflect">
     <link name="${prefix}_ezgripper_finger_L2_${postfix}">
       <visual>
@@ -80,7 +80,7 @@
       </inertial>
     </link>
-</macro>
+</xacro:macro>
     <!-- joints -->
-<macro name="ezgripper_knuckle_palm_L1" params="prefix postfix reflectY reflectZ reflectR mimic_test">
+<xacro:macro name="ezgripper_knuckle_palm_L1" params="prefix postfix reflectY reflectZ reflectR mimic_test">
     <joint name="${prefix}_ezgripper_knuckle_palm_L1_${postfix}" type="revolute">
       <parent link="${prefix}_ezgripper_palm_link"/>
@@ -93,6 +93,6 @@
       </xacro:if>
     </joint>
-</macro>
-<macro name="ezgripper_knuckle_L1_L2" params="prefix postfix reflectY reflectZ reflectR mimic_test">
+</xacro:macro>
+<xacro:macro name="ezgripper_knuckle_L1_L2" params="prefix postfix reflectY reflectZ reflectR mimic_test">
     <joint name="${prefix}_ezgripper_knuckle_L1_L2_${postfix}" type="revolute">
       <parent link="${prefix}_ezgripper_finger_L1_${postfix}"/>
@@ -106,7 +106,7 @@
       </xacro:if>
     </joint>
-</macro>
+</xacro:macro>
     <!-- transmissions for Gazebo -->
-<macro name="ezgripper_knuckle_trans" params="prefix postfix">
+<xacro:macro name="ezgripper_knuckle_trans" params="prefix postfix">
    <transmission name="${prefix}_ezgripper_trans_${postfix}">
       <type>transmission_interface/SimpleTransmission</type>
@@ -119,6 +119,6 @@
       </actuator>
    </transmission>
-</macro>
-<macro name="gazebo_knuckle_jsp" params="prefix">
+</xacro:macro>
+<xacro:macro name="gazebo_knuckle_jsp" params="prefix">
    <gazebo>
      <plugin name="joint_state_publisher" filename="libgazebo_ros_joint_state_publisher.so">
@@ -126,5 +126,5 @@
      </plugin>
    </gazebo>
-</macro>
+</xacro:macro>
 <gazebo>
    <plugin name="gazebo_ros_control" filename="libgazebo_ros_control.so">
