Commit message: Fixed passing of origin into ezgripper_dual_articulated.urdf.xacro

File: ezgripper_driver/urdf/ezgripper_dual_gen2_standalone.urdf.xacro (robot description, xacro)
@@ -1,7 +1,7 @@
 <?xml version="1.0" encoding="UTF-8"?>
 <robot name="ezgripper_stand_alone" xmlns:xacro="http://www.ros.org/wiki/xacro">
-<property name="ezgripper_offset_x" value="0.049"/>
+<property name="ezgripper_offset_x" value="0.0"/>
 <property name="ezgripper_offset_y" value="0.0"/>
-<property name="ezgripper_offset_z" value="0.21"/>
+<property name="ezgripper_offset_z" value="0.0"/>
 <xacro:include filename="$(find ezgripper_driver)/urdf/ezgripper_dual_gen2_articulated.urdf.xacro"/>
 <!-- Add the gripper -->
@@ -19,5 +19,5 @@
            <cylinder length="0.42" radius="0.02"/>
         </geometry>
-        <origin rpy="0 0 0" xyz="0 0 0.21"/>
+        <origin rpy="0 0 0" xyz="0 0 0.0"/>
         <material name="red"/>
     </visual>

Commit message: fix xacro warnings

File: ezgripper_driver/urdf/ezgripper_dual_gen2_standalone.urdf.xacro (robot description, xacro)
@@ -1,7 +1,7 @@
 <?xml version="1.0" encoding="UTF-8"?>
-<robot name="ezgripper_stand_alone" xmlns:xacro="http://www.ros.org/wiki/xacro">
-<property name="ezgripper_offset_x" value="0.0"/>
-<property name="ezgripper_offset_y" value="0.0"/>
-<property name="ezgripper_offset_z" value="0.0"/>
+<robot name="ezgripper_stand_alone" xmlns:xacro="http://ros.org/wiki/xacro">
+<xacro:property name="ezgripper_offset_x" value="0.0"/>
+<xacro:property name="ezgripper_offset_y" value="0.0"/>
+<xacro:property name="ezgripper_offset_z" value="0.0"/>
 <xacro:include filename="$(find ezgripper_driver)/urdf/ezgripper_dual_gen2_articulated.urdf.xacro"/>
 <!-- Add the gripper -->

File: ezgripper_driver/urdf/ezgripper_dual_standalone.urdf.xacro (robot description, xacro)
@@ -1,7 +1,7 @@
 <?xml version="1.0" encoding="UTF-8"?>
-<robot name="ezgripper_stand_alone" xmlns:xacro="http://www.ros.org/wiki/xacro">
-<property name="ezgripper_offset_x" value="0.049"/>
-<property name="ezgripper_offset_y" value="0.0"/>
-<property name="ezgripper_offset_z" value="0.21"/>
+<robot name="ezgripper_stand_alone" xmlns:xacro="http://ros.org/wiki/xacro">
+<xacro:property name="ezgripper_offset_x" value="0.049"/>
+<xacro:property name="ezgripper_offset_y" value="0.0"/>
+<xacro:property name="ezgripper_offset_z" value="0.21"/>
 <xacro:include filename="$(find ezgripper_driver)/urdf/ezgripper_dual.urdf.xacro"/>
 <!-- Add the gripper -->

File: ezgripper_driver/urdf/ezgripper_quad_standalone.urdf.xacro (robot description, xacro)
@@ -1,7 +1,7 @@
 <?xml version="1.0" encoding="UTF-8"?>
-<robot name="ezgripper_stand_alone" xmlns:xacro="http://www.ros.org/wiki/xacro">
-<property name="ezgripper_offset_x" value="0.049"/>
-<property name="ezgripper_offset_y" value="0.0"/>
-<property name="ezgripper_offset_z" value="0.21"/>
+<robot name="ezgripper_stand_alone" xmlns:xacro="http://ros.org/wiki/xacro">
+<xacro:property name="ezgripper_offset_x" value="0.049"/>
+<xacro:property name="ezgripper_offset_y" value="0.0"/>
+<xacro:property name="ezgripper_offset_z" value="0.21"/>
 <xacro:include filename="$(find ezgripper_driver)/urdf/ezgripper_quad.urdf.xacro"/>
 <!-- Add the gripper -->
