Commit message: software fix

File: ezgripper_driver/urdf/dual_gen1/ezgripper_dual_gen1.urdf.xacro (robot description, xacro)
@@ -1,6 +1,5 @@
 <?xml version="1.0" encoding="UTF-8"?>
 <robot name="ezgripper" xmlns:xacro="http://ros.org/wiki/xacro">
-<!--macro name="ezgripper" params="*origin"-->
-<xacro:macro name="ezgripper_dual_gen2" params="prefix parent_link *origin">
+<xacro:macro name="ezgripper_dual_gen1" params="prefix parent_link *origin">
     <!-- links -->
     <link name="${prefix}_ezgripper_palm_link">
@@ -8,11 +7,12 @@
         <origin xyz="0 0 0" rpy="0 0 0"/>
         <geometry>
-          <mesh filename="package://ezgripper_driver/meshes/visual/SAKE_Palm_Dual_Gen2.stl"/>
+          <mesh filename="package://ezgripper_driver/meshes/dual_gen1/SAKE_Palm_Dual.stl"/>
         </geometry>
+				<material name="blue"/>
       </visual>
       <collision>
         <origin xyz="0 0 0" rpy="0 0 0"/>
         <geometry>
-          <mesh filename="package://ezgripper_driver/meshes/collision/SAKE_Palm_Dual_Gen2.stl"/>
+          <mesh filename="package://ezgripper_driver/meshes/dual_gen1/SAKE_Palm_Dual.stl"/>
         </geometry>
       </collision>
@@ -22,6 +22,9 @@
     </inertial>
     </link>
+		<gazebo reference="${prefix}_ezgripper_palm_link">
+      <material>Gazebo/Blue</material>
+   </gazebo>
     <joint name="${prefix}_ezgripper_connect" type="fixed">
-        <origin rpy="-1.57 0 0" xyz="0.049 0.0 0.2"/>
+				<xacro:insert_block name="origin" />
         <parent link="${parent_link}"/>
         <child link="${prefix}_ezgripper_palm_link"/>
@@ -31,6 +34,7 @@
     <ezgripper_finger prefix="${prefix}" postfix="1" reflect="1" />
     <ezgripper_finger prefix="${prefix}" postfix="2" reflect="1" />
+		<!-- Mimic Test has to set false for the first joint -->
     <ezgripper_knuckle prefix="${prefix}" postfix="1" reflectY="1" reflectZ="1" reflectR="1" mimic_test="false"/>
-    <ezgripper_knuckle prefix="${prefix}" postfix="2" reflectY="-1" reflectZ="1" reflectR="-1" mimic_test="true"/>
+    <ezgripper_knuckle prefix="${prefix}" postfix="2" reflectY="-1" reflectZ="1" reflectR="-1" mimic_test="false"/>
     <ezgripper_knuckle_trans prefix="${prefix}" postfix="1"/>
     <ezgripper_knuckle_trans prefix="${prefix}" postfix="2"/>
@@ -42,11 +46,12 @@
         <origin xyz="0 0 0" rpy="0 0 0"/>
         <geometry>
-          <mesh filename="package://ezgripper_driver/meshes/visual/SAKE_Finger_Gen2.stl"/>
+          <mesh filename="package://ezgripper_driver/meshes/dual_gen1/SAKE_Finger.stl"/>
         </geometry>
+				<material name="grey"/>
       </visual>
       <collision>
         <origin xyz="0 0 0" rpy="0 0 0"/>
         <geometry>
-          <mesh filename="package://ezgripper_driver/meshes/collision/SAKE_Finger_Gen2.stl"/>
+          <mesh filename="package://ezgripper_driver/meshes/dual_gen1/SAKE_Finger.stl"/>
         </geometry>
       </collision>
@@ -56,4 +61,7 @@
       </inertial>
     </link>
+		<gazebo reference="${prefix}_ezgripper_finger_${postfix}">
+      <material>Gazebo/Grey</material>
+   </gazebo>
 </xacro:macro>
     <!-- joints -->
@@ -66,5 +74,5 @@
       <limit lower="-.27" upper="1.57075" effort="1" velocity="3.67"/>
       <xacro:if value="${mimic_test}">
-           <mimic joint="ezgripper_knuckle_1"/>
+           <mimic joint="${prefix}_ezgripper_knuckle_1"/>
       </xacro:if>
     </joint>
@@ -75,9 +83,9 @@
       <type>transmission_interface/SimpleTransmission</type>
       <joint name="${prefix}_ezgripper_knuckle_${postfix}">
-         <hardwareInterface>PositionJointInterface</hardwareInterface>
+         <hardwareInterface>hardware_interface/PositionJointInterface</hardwareInterface>
       </joint>
       <actuator name="${prefix}_ezgripper_motor${postfix}">
          <mechanicalReduction>1</mechanicalReduction>
-         <hardwareInterface>PositionJointInterface</hardwareInterface>
+         <hardwareInterface>hardware_interface/PositionJointInterface</hardwareInterface>
       </actuator>
    </transmission>
@@ -86,5 +94,5 @@
    <gazebo>
      <plugin name="joint_state_publisher" filename="libgazebo_ros_joint_state_publisher.so">
-       <jointName>${prefix}_ezgripper_knuckle_1,${prefix}_ezgripper_knuckle_2  </jointName>
+       <jointName>${prefix}_ezgripper_knuckle_1,${prefix}_ezgripper_knuckle_2 </jointName>
      </plugin>
    </gazebo>
@@ -92,4 +100,5 @@
 <gazebo>
    <plugin name="gazebo_ros_control" filename="libgazebo_ros_control.so">
+		<legacyModeNS>true</legacyModeNS>
    </plugin>
 </gazebo>

File: ezgripper_driver/urdf/dual_gen2/ezgripper_dual_gen2_articulated.urdf.xacro (robot description, xacro)
@@ -1,6 +1,5 @@
 <?xml version="1.0" encoding="UTF-8"?>
 <robot name="ezgripper" xmlns:xacro="http://ros.org/wiki/xacro">
-<!--macro name="ezgripper" params="*origin"-->
-<xacro:macro name="ezgripper_dual" params="prefix parent_link *origin">
+<xacro:macro name="ezgripper_dual_gen2" params="prefix parent_link *origin">
     <!-- links -->
     <link name="${prefix}_ezgripper_palm_link">
@@ -8,11 +7,12 @@
         <origin xyz="0 0 0" rpy="0 0 0"/>
         <geometry>
-          <mesh filename="package://ezgripper_driver/meshes/visual/SAKE_Palm_Dual.stl"/>
+          <mesh filename="package://ezgripper_driver/meshes/dual_gen2/SAKE_Palm_Dual_Gen2.stl"/>
         </geometry>
+				<material name="blue"/>
       </visual>
       <collision>
         <origin xyz="0 0 0" rpy="0 0 0"/>
         <geometry>
-          <mesh filename="package://ezgripper_driver/meshes/collision/SAKE_Palm_Dual.stl"/>
+          <mesh filename="package://ezgripper_driver/meshes/dual_gen2/SAKE_Palm_Dual_Gen2.stl"/>
         </geometry>
       </collision>
@@ -22,6 +22,9 @@
     </inertial>
     </link>
+		<gazebo reference="${prefix}_ezgripper_palm_link">
+      <material>Gazebo/Blue</material>
+   </gazebo>
     <joint name="${prefix}_ezgripper_connect" type="fixed">
-        <origin rpy="-1.57 0 0" xyz="0.049 0.0 0.2"/>
+        <xacro:insert_block name="origin" />
         <parent link="${parent_link}"/>
         <child link="${prefix}_ezgripper_palm_link"/>
@@ -33,10 +36,13 @@
     <ezgripper_finger_L2 prefix="${prefix}" postfix="1" reflect="1" />
     <ezgripper_finger_L2 prefix="${prefix}" postfix="2" reflect="1" />
+		<!-- Mimic Test has to set false for the first joint -->
     <ezgripper_knuckle_palm_L1 prefix="${prefix}" postfix="1" reflectY="1" reflectZ="1" reflectR="1" mimic_test="false"/>
-    <ezgripper_knuckle_palm_L1 prefix="${prefix}" postfix="2" reflectY="-1" reflectZ="1" reflectR="-1" mimic_test="true"/>
-    <ezgripper_knuckle_L1_L2 prefix="${prefix}" postfix="1" reflectY="1" reflectZ="1" reflectR="1" mimic_test="false"/>
-    <ezgripper_knuckle_L1_L2 prefix="${prefix}" postfix="2" reflectY="-1" reflectZ="1" reflectR="-1" mimic_test="true"/>
-    <ezgripper_knuckle_trans prefix="${prefix}" postfix="1"/>
-    <ezgripper_knuckle_trans prefix="${prefix}" postfix="2"/>
+    <ezgripper_knuckle_palm_L1 prefix="${prefix}" postfix="2" reflectY="-1" reflectZ="1" reflectR="-1" mimic_test="false"/>
+    <ezgripper_knuckle_L1_L2 prefix="${prefix}" postfix="1" reflectY="1" reflectZ="1" reflectR="-1" mimic_test="false"/>
+    <ezgripper_knuckle_L1_L2 prefix="${prefix}" postfix="2" reflectY="-1" reflectZ="1" reflectR="1" mimic_test="false"/>
+		<ezgripper_knuckle_palm_trans prefix="${prefix}" postfix="L1_1"/>
+		<ezgripper_knuckle_palm_trans prefix="${prefix}" postfix="L1_2"/>
+    <ezgripper_knuckle_trans prefix="${prefix}" postfix="L1_L2_1"/>
+		<ezgripper_knuckle_trans prefix="${prefix}" postfix="L1_L2_2"/>
     <gazebo_knuckle_jsp prefix="${prefix}" />
 </xacro:macro>
@@ -46,11 +52,12 @@
         <origin xyz="0 0 0" rpy="0 0 0"/>
         <geometry>
-          <mesh filename="package://ezgripper_driver/meshes/visual/SAKE_Finger_L1.stl"/>
+          <mesh filename="package://ezgripper_driver/meshes/dual_gen2/SAKE_Finger_L1_Gen2.stl"/>
         </geometry>
+				<material name="grey"/>
       </visual>
       <collision>
         <origin xyz="0 0 0" rpy="0 0 0"/>
         <geometry>
-          <mesh filename="package://ezgripper_driver/meshes/collision/SAKE_Finger_L1.stl"/>
+          <mesh filename="package://ezgripper_driver/meshes/dual_gen2/SAKE_Finger_L1_Gen2.stl"/>
         </geometry>
       </collision>
@@ -60,4 +67,7 @@
       </inertial>
     </link>
+		<gazebo reference="${prefix}_ezgripper_finger_L1_${postfix}">
+      <material>Gazebo/Grey</material>
+   </gazebo>
 </xacro:macro>
 <xacro:macro name="ezgripper_finger_L2" params="prefix postfix reflect">
@@ -66,11 +76,12 @@
         <origin xyz="0 0 0" rpy="0 0 0"/>
         <geometry>
-          <mesh filename="package://ezgripper_driver/meshes/visual/SAKE_Finger_L2.stl"/>
+          <mesh filename="package://ezgripper_driver/meshes/dual_gen2/SAKE_Finger_L2_Gen2.stl"/>
         </geometry>
+				<material name="grey"/>
       </visual>
       <collision>
         <origin xyz="0 0 0" rpy="0 0 0"/>
         <geometry>
-          <mesh filename="package://ezgripper_driver/meshes/collision/SAKE_Finger_L2.stl"/>
+          <mesh filename="package://ezgripper_driver/meshes/dual_gen2/SAKE_Finger_L2_Gen2.stl"/>
         </geometry>
       </collision>
@@ -80,4 +91,7 @@
       </inertial>
     </link>
+		<gazebo reference="${prefix}_ezgripper_finger_L2_${postfix}">
+      <material>Gazebo/Grey</material>
+   </gazebo>
 </xacro:macro>
     <!-- joints -->
@@ -86,7 +100,7 @@
       <parent link="${prefix}_ezgripper_palm_link"/>
       <child link="${prefix}_ezgripper_finger_L1_${postfix}"/>
-      <origin xyz="0.1056 ${reflectY*0.03} 0" rpy="${1.5708 * reflectR} 0 3.14159"/>
+      <origin xyz="0.072569 ${reflectY*0.03} 0" rpy="${-1.5708 * reflectR} 0 ${1.57075 * reflectR}"/>
       <axis xyz="0 1 0"/>
-      <limit lower="-.27" upper="1.57075" effort="1" velocity="3.67"/>
+      <limit lower="0" upper="1.94" effort="1" velocity="3.67"/>
       <xacro:if value="${mimic_test}">
            <mimic joint="${prefix}_ezgripper_knuckle_palm_L1_1"/>
@@ -98,7 +112,8 @@
       <parent link="${prefix}_ezgripper_finger_L1_${postfix}"/>
       <child link="${prefix}_ezgripper_finger_L2_${postfix}"/>
-      <origin xyz="0.1056 ${reflectY*0.03} 0" rpy="${1.5708 * reflectR} 0 3.14159"/>
+      <origin xyz="0.052 0 0" rpy="0 0 0"/>
+      <!-- origin xyz="0.06 0 0" rpy="${3.14159 * reflectR} 0 0"/-->
       <axis xyz="0 1 0"/>
-      <limit lower="-.27" upper="1.57075" effort="1" velocity="3.67"/>
+      <limit lower="0" upper="1.94" effort="1" velocity="3.67"/>
       <xacro:if value="${mimic_test}">
            <mimic joint="${prefix}_ezgripper_knuckle_L1_L2_1"/>
@@ -107,13 +122,25 @@
 </xacro:macro>
     <!-- transmissions for Gazebo -->
+<xacro:macro name="ezgripper_knuckle_palm_trans" params="prefix postfix">
+	<transmission name="${prefix}_ezgripper_knuckle_palm_trans_${postfix}">
+			<type>transmission_interface/SimpleTransmission</type>
+			<joint name="${prefix}_ezgripper_knuckle_palm_${postfix}">
+				<hardwareInterface>hardware_interface/PositionJointInterface</hardwareInterface>
+			</joint>
+			<actuator name="${prefix}_ezgripper_knuckle_palm_motor${postfix}">
+				<mechanicalReduction>1</mechanicalReduction>
+				<hardwareInterface>hardware_interface/PositionJointInterface</hardwareInterface>
+			</actuator>
+	</transmission>
+</xacro:macro>
 <xacro:macro name="ezgripper_knuckle_trans" params="prefix postfix">
-   <transmission name="${prefix}_ezgripper_trans_${postfix}">
+   <transmission name="${prefix}_ezgripper_knuckle_trans_${postfix}">
       <type>transmission_interface/SimpleTransmission</type>
       <joint name="${prefix}_ezgripper_knuckle_${postfix}">
-         <hardwareInterface>PositionJointInterface</hardwareInterface>
+         <hardwareInterface>hardware_interface/PositionJointInterface</hardwareInterface>
       </joint>
-      <actuator name="${prefix}_ezgripper_motor${postfix}">
+      <actuator name="${prefix}_ezgripper_knuckle_motor${postfix}">
          <mechanicalReduction>1</mechanicalReduction>
-         <hardwareInterface>PositionJointInterface</hardwareInterface>
+         <hardwareInterface>hardware_interface/PositionJointInterface</hardwareInterface>
       </actuator>
    </transmission>
@@ -122,5 +149,5 @@
    <gazebo>
      <plugin name="joint_state_publisher" filename="libgazebo_ros_joint_state_publisher.so">
-       <jointName>${prefix}_ezgripper_knuckle_1,${prefix}_ezgripper_knuckle_2  </jointName>
+       <jointName>${prefix}_ezgripper_knuckle_palm_L1_1,${prefix}_ezgripper_knuckle_palm_L1_2,${prefix}_ezgripper_knuckle_L1_L2_1,${prefix}_ezgripper_knuckle_L1_L2_2</jointName>
      </plugin>
    </gazebo>
@@ -128,4 +155,5 @@
 <gazebo>
    <plugin name="gazebo_ros_control" filename="libgazebo_ros_control.so">
+		<legacyModeNS>true</legacyModeNS>
    </plugin>
 </gazebo>

File: ezgripper_driver/urdf/quad/ezgripper_quad.urdf.xacro (robot description, xacro)
@@ -7,11 +7,12 @@
         <origin xyz="0 0 0" rpy="0 0 0"/>
         <geometry>
-          <mesh filename="package://ezgripper_driver/meshes/visual/SAKE_Palm_Quad.stl"/>
+          <mesh filename="package://ezgripper_driver/meshes/quad/SAKE_Palm_Quad.stl"/>
         </geometry>
+				<material name="blue"/>
       </visual>
       <collision>
         <origin xyz="0 0 0" rpy="0 0 0"/>
         <geometry>
-          <mesh filename="package://ezgripper_driver/meshes/collision/SAKE_Palm_Quad.stl"/>
+          <mesh filename="package://ezgripper_driver/meshes/quad/SAKE_Palm_Quad.stl"/>
         </geometry>
       </collision>
@@ -21,6 +22,9 @@
     </inertial>
     </link>
+		<gazebo reference="${prefix}_ezgripper_palm_link">
+      <material>Gazebo/Blue</material>
+   </gazebo>
     <joint name="${prefix}_ezgripper_connect" type="fixed">
-        <origin rpy="-1.57 0 0" xyz="0.049 0.0 0.2"/>
+				<xacro:insert_block name="origin" />
         <parent link="${parent_link}"/>
         <child link="${prefix}_ezgripper_palm_link"/>
@@ -28,17 +32,18 @@
         <limit effort="0" lower="-1.57075" upper="0.25" velocity="3.67"/>
     </joint>
-    <ezgripper_finger prefix="${prefix}" postfix="1" reflect="1"/>
-    <ezgripper_finger prefix="${prefix}" postfix="2" reflect="1"/>
-    <ezgripper_finger prefix="${prefix}" postfix="3" reflect="1"/>
-    <ezgripper_finger prefix="${prefix}" postfix="4" reflect="1"/>
-    <ezgripper_knuckle prefix="${prefix}" postfix="1" reflectY="1" reflectZ="1" reflectR="1" mimic_test="false"/>
-    <ezgripper_knuckle prefix="${prefix}" postfix="2" reflectY="-1" reflectZ="1" reflectR="-1" mimic_test="true"/>
-    <ezgripper_knuckle prefix="${prefix}" postfix="3" reflectY="1" reflectZ="-1" reflectR="1" mimic_test="true"/>
-    <ezgripper_knuckle prefix="${prefix}" postfix="4" reflectY="-1" reflectZ="-1" reflectR="-1" mimic_test="true"/>
-    <ezgripper_knuckle_trans prefix="${prefix}" postfix="1"/>
-    <ezgripper_knuckle_trans prefix="${prefix}" postfix="2"/>
-    <ezgripper_knuckle_trans prefix="${prefix}" postfix="3"/>
-    <ezgripper_knuckle_trans prefix="${prefix}" postfix="4"/>
-    <gazebo_knuckle_jsp prefix="${prefix}" />
+    <xacro:ezgripper_finger prefix="${prefix}" postfix="1" reflect="1"/>
+    <xacro:ezgripper_finger prefix="${prefix}" postfix="2" reflect="1"/>
+    <xacro:ezgripper_finger prefix="${prefix}" postfix="3" reflect="1"/>
+    <xacro:ezgripper_finger prefix="${prefix}" postfix="4" reflect="1"/>
+		<!-- Mimic Test has to set false for the first joint -->
+    <xacro:ezgripper_knuckle prefix="${prefix}" postfix="1" reflectY="1" reflectZ="1" reflectR="1" mimic_test="false"/>
+    <xacro:ezgripper_knuckle prefix="${prefix}" postfix="2" reflectY="-1" reflectZ="1" reflectR="-1" mimic_test="false"/>
+    <xacro:ezgripper_knuckle prefix="${prefix}" postfix="3" reflectY="1" reflectZ="-1" reflectR="1" mimic_test="false"/>
+    <xacro:ezgripper_knuckle prefix="${prefix}" postfix="4" reflectY="-1" reflectZ="-1" reflectR="-1" mimic_test="false"/>
+    <xacro:ezgripper_knuckle_trans prefix="${prefix}" postfix="1"/>
+    <xacro:ezgripper_knuckle_trans prefix="${prefix}" postfix="2"/>
+    <xacro:ezgripper_knuckle_trans prefix="${prefix}" postfix="3"/>
+    <xacro:ezgripper_knuckle_trans prefix="${prefix}" postfix="4"/>
+    <xacro:gazebo_knuckle_jsp prefix="${prefix}" />
 </xacro:macro>
 <xacro:macro name="ezgripper_finger" params="prefix postfix reflect">
@@ -47,11 +52,12 @@
         <origin xyz="0 0 0" rpy="0 0 0"/>
         <geometry>
-          <mesh filename="package://ezgripper_driver/meshes/visual/SAKE_Finger.stl"/>
+          <mesh filename="package://ezgripper_driver/meshes/quad/SAKE_Finger.stl"/>
         </geometry>
+				<material name="grey"/>
       </visual>
       <collision>
         <origin xyz="0 0 0" rpy="0 0 0"/>
         <geometry>
-          <mesh filename="package://ezgripper_driver/meshes/collision/SAKE_Finger.stl"/>
+          <mesh filename="package://ezgripper_driver/meshes/quad/SAKE_Finger.stl"/>
         </geometry>
       </collision>
@@ -61,6 +67,9 @@
       </inertial>
     </link>
+		<gazebo reference="${prefix}_ezgripper_finger_${postfix}">
+      <material>Gazebo/Grey</material>
+   </gazebo>
 </xacro:macro>
-    <!-- joints -->
+<!-- joints -->
 <xacro:macro name="ezgripper_knuckle" params="prefix postfix reflectY reflectZ reflectR mimic_test">
     <joint name="${prefix}_ezgripper_knuckle_${postfix}" type="revolute">
@@ -80,9 +89,9 @@
       <type>transmission_interface/SimpleTransmission</type>
       <joint name="${prefix}_ezgripper_knuckle_${postfix}">
-         <hardwareInterface>PositionJointInterface</hardwareInterface>
+         <hardwareInterface>hardware_interface/PositionJointInterface</hardwareInterface>
       </joint>
       <actuator name="${prefix}_ezgripper_motor${postfix}">
          <mechanicalReduction>1</mechanicalReduction>
-         <hardwareInterface>PositionJointInterface</hardwareInterface>
+         <hardwareInterface>hardware_interface/PositionJointInterface</hardwareInterface>
       </actuator>
    </transmission>
@@ -97,4 +106,5 @@
 <gazebo>
    <plugin name="gazebo_ros_control" filename="libgazebo_ros_control.so">
+		<legacyModeNS>true</legacyModeNS>
    </plugin>
 </gazebo>
