Commit message: shifted to GripperAction

File: ezgripper_driver/urdf/dual_gen1/ezgripper_dual_gen1_standalone.urdf.xacro (robot description, xacro)
@@ -23,4 +23,10 @@
         <material name="black"/>
     </visual>
+		<collision>
+			<geometry>
+					<cylinder length="0.42" radius="0.02"/>
+			 </geometry>
+			 <origin rpy="0 0 0" xyz="0 0 0.21"/>
+		</collision>
 </link>
 <gazebo reference="base_link">

File: ezgripper_driver/urdf/dual_gen2/ezgripper_dual_gen2_articulated.urdf.xacro (robot description, xacro)
@@ -38,11 +38,12 @@
 		<!-- Mimic Test has to set false for the first joint -->
     <xacro:ezgripper_knuckle_palm_L1 prefix="${prefix}" postfix="1" reflectY="1" reflectZ="1" reflectR="1" mimic_test="false"/>
-    <xacro:ezgripper_knuckle_palm_L1 prefix="${prefix}" postfix="2" reflectY="-1" reflectZ="1" reflectR="-1" mimic_test="false"/>
+    <xacro:ezgripper_knuckle_palm_L1 prefix="${prefix}" postfix="2" reflectY="-1" reflectZ="1" reflectR="-1" mimic_test="true"/>
     <xacro:ezgripper_knuckle_L1_L2 prefix="${prefix}" postfix="1" reflectY="1" reflectZ="1" reflectR="-1" mimic_test="false"/>
-    <xacro:ezgripper_knuckle_L1_L2 prefix="${prefix}" postfix="2" reflectY="-1" reflectZ="1" reflectR="1" mimic_test="false"/>
+    <xacro:ezgripper_knuckle_L1_L2 prefix="${prefix}" postfix="2" reflectY="-1" reflectZ="1" reflectR="1" mimic_test="true"/>
+		<!-- Transmission needs to be removed when mimicked -->
 		<xacro:ezgripper_knuckle_palm_trans prefix="${prefix}" postfix="L1_1"/>
-		<xacro:ezgripper_knuckle_palm_trans prefix="${prefix}" postfix="L1_2"/>
+		<!-- <xacro:ezgripper_knuckle_palm_trans prefix="${prefix}" postfix="L1_2"/> -->
     <xacro:ezgripper_knuckle_trans prefix="${prefix}" postfix="L1_L2_1"/>
-		<xacro:ezgripper_knuckle_trans prefix="${prefix}" postfix="L1_L2_2"/>
+		<!-- <xacro:ezgripper_knuckle_trans prefix="${prefix}" postfix="L1_L2_2"/> -->
     <xacro:gazebo_knuckle_jsp prefix="${prefix}" />
 </xacro:macro>
@@ -157,4 +158,9 @@
 		<legacyModeNS>true</legacyModeNS>
    </plugin>
+	 <!-- Fix mimicking bug -->
+	 <plugin filename="libroboticsgroup_upatras_gazebo_mimic_joint_plugin.so" name="mimicker">
+		<joint>left_ezgripper_knuckle_palm_L1_1</joint>
+		<mimicJoint>left_ezgripper_knuckle_palm_L1_2</mimicJoint>
+	</plugin>
 </gazebo>
 </robot>

File: ezgripper_driver/urdf/dual_gen2/ezgripper_dual_gen2_standalone.urdf.xacro (robot description, xacro)
@@ -23,4 +23,10 @@
         <material name="black"/>
     </visual>
+		<collision>
+			<geometry>
+					<cylinder length="0.42" radius="0.02"/>
+			 </geometry>
+			 <origin rpy="0 0 0" xyz="0 0 0.21"/>
+		</collision>
 </link>
 <gazebo reference="base_link">

File: ezgripper_driver/urdf/quad/ezgripper_quad_standalone.urdf.xacro (robot description, xacro)
@@ -23,4 +23,10 @@
         <material name="black"/>
     </visual>
+		<collision>
+			<geometry>
+					<cylinder length="0.42" radius="0.02"/>
+			 </geometry>
+			 <origin rpy="0 0 0" xyz="0 0 0.21"/>
+		</collision>
 </link>
 <gazebo reference="base_link">
