Commit message: fixing max effort

File: ezgripper_driver/urdf/dual_gen2/ezgripper_dual_gen2_articulated.urdf.xacro (robot description, xacro)
@@ -103,5 +103,5 @@
       <origin xyz="0.072569 ${reflectY*0.03} 0" rpy="${-1.5708 * reflectR} 0 ${1.57075 * reflectR}"/>
       <axis xyz="0 1 0"/>
-      <limit lower="0" upper="1.94" effort="1" velocity="3.67"/>
+      <limit lower="0" upper="1.94" effort="100" velocity="3.67"/>
       <xacro:if value="${mimic_test}">
            <mimic joint="${prefix}_ezgripper_knuckle_palm_L1_1"/>
@@ -116,5 +116,5 @@
       <!-- origin xyz="0.06 0 0" rpy="${3.14159 * reflectR} 0 0"/-->
       <axis xyz="0 1 0"/>
-      <limit lower="0" upper="1.94" effort="1" velocity="3.67"/>
+      <limit lower="0" upper="1.94" effort="100" velocity="3.67"/>
       <xacro:if value="${mimic_test}">
            <mimic joint="${prefix}_ezgripper_knuckle_L1_L2_1"/>

Commit message: increased joint limits

File: ezgripper_driver/urdf/dual_gen2/ezgripper_dual_gen2_articulated.urdf.xacro (robot description, xacro)
@@ -100,5 +100,5 @@
 				<origin xyz="0.072569 ${reflectY*0.03} 0" rpy="${-1.5708 * reflectR} 0 ${1.57075 * reflectR}"/>
 				<axis xyz="0 1 0"/>
-				<limit lower="0" upper="1.92" effort="1.0" velocity="3.67"/>
+				<limit lower="0" upper="1.94" effort="1.0" velocity="3.67"/>
 				<xacro:if value="${mimic_test}">
 						<mimic joint="${prefix}_ezgripper_knuckle_palm_L1_1"/>
