Commit message: reorganised package structure

File: ezgripper_description/urdf/dual_gen1/ezgripper_dual_gen1.urdf.xacro (robot description, xacro)
@@ -1,5 +1,5 @@
 <?xml version="1.0" encoding="UTF-8"?>
-<robot name="ezgripper_quad" xmlns:xacro="http://ros.org/wiki/xacro">
-	<xacro:macro name="ezgripper_quad" params="prefix parent_link *origin">
+<robot name="ezgripper_dual_gen1" xmlns:xacro="http://ros.org/wiki/xacro">
+	<xacro:macro name="ezgripper_dual_gen1" params="prefix parent_link *origin">
 			<!-- links -->
 			<link name="${prefix}_ezgripper_palm_link">
@@ -7,5 +7,5 @@
 					<origin xyz="0 0 0" rpy="0 0 0"/>
 					<geometry>
-						<mesh filename="package://ezgripper_driver/meshes/quad/SAKE_Palm_Quad.stl"/>
+						<mesh filename="package://ezgripper_description/meshes/dual_gen1/SAKE_Palm_Dual.stl"/>
 					</geometry>
 					<material name="blue"/>
@@ -14,5 +14,5 @@
 					<origin xyz="0 0 0" rpy="0 0 0"/>
 					<geometry>
-						<mesh filename="package://ezgripper_driver/meshes/quad/SAKE_Palm_Quad.stl"/>
+						<mesh filename="package://ezgripper_description/meshes/dual_gen1/SAKE_Palm_Dual.stl"/>
 					</geometry>
 				</collision>
@@ -32,18 +32,12 @@
 					<limit effort="0" lower="-1.57075" upper="0.25" velocity="3.67"/>
 			</joint>
-			<xacro:ezgripper_finger prefix="${prefix}" postfix="1" reflect="1"/>
-			<xacro:ezgripper_finger prefix="${prefix}" postfix="2" reflect="1"/>
-			<xacro:ezgripper_finger prefix="${prefix}" postfix="3" reflect="1"/>
-			<xacro:ezgripper_finger prefix="${prefix}" postfix="4" reflect="1"/>
-			<!-- Mimic Test has to be set false for the first joint -->
+			<xacro:ezgripper_finger prefix="${prefix}" postfix="1" reflect="1" />
+			<xacro:ezgripper_finger prefix="${prefix}" postfix="2" reflect="1" />
+			<!-- Mimic Test has to set be false for the first joint -->
 			<xacro:ezgripper_knuckle prefix="${prefix}" postfix="1" reflectY="1" reflectZ="1" reflectR="1" mimic_test="false"/>
 			<xacro:ezgripper_knuckle prefix="${prefix}" postfix="2" reflectY="-1" reflectZ="1" reflectR="-1" mimic_test="true"/>
-			<xacro:ezgripper_knuckle prefix="${prefix}" postfix="3" reflectY="1" reflectZ="-1" reflectR="1" mimic_test="true"/>
-			<xacro:ezgripper_knuckle prefix="${prefix}" postfix="4" reflectY="-1" reflectZ="-1" reflectR="-1" mimic_test="true"/>
 			<!-- Transmission needs to be removed when mimicked -->
 			<xacro:ezgripper_knuckle_trans prefix="${prefix}" postfix="1"/>
-			<!-- <xacro:ezgripper_knuckle_trans prefix="${prefix}" postfix="2"/>
-			<xacro:ezgripper_knuckle_trans prefix="${prefix}" postfix="3"/>
-			<xacro:ezgripper_knuckle_trans prefix="${prefix}" postfix="4"/> -->
+			<!-- <xacro:ezgripper_knuckle_trans prefix="${prefix}" postfix="2"/> -->
 			<xacro:gazebo_knuckle_jsp prefix="${prefix}" />
 	</xacro:macro>
@@ -53,5 +47,5 @@
 					<origin xyz="0 0 0" rpy="0 0 0"/>
 					<geometry>
-						<mesh filename="package://ezgripper_driver/meshes/quad/SAKE_Finger.stl"/>
+						<mesh filename="package://ezgripper_description/meshes/dual_gen1/SAKE_Finger.stl"/>
 					</geometry>
 					<material name="grey"/>
@@ -60,10 +54,10 @@
 					<origin xyz="0 0 0" rpy="0 0 0"/>
 					<geometry>
-						<mesh filename="package://ezgripper_driver/meshes/quad/SAKE_Finger.stl"/>
+						<mesh filename="package://ezgripper_description/meshes/dual_gen1/SAKE_Finger.stl"/>
 					</geometry>
 				</collision>
 				<inertial>
 					<mass value=".025"/>
-					<inertia ixx="0.01" ixy="0.0" ixz="0.0" iyy=".01" iyz="0.0" izz="0.01"/>
+					<inertia ixx="0.01" ixy="0.0" ixz="0.0" iyy="0.01" iyz="0.0" izz="0.01"/>
 				</inertial>
 			</link>
@@ -77,5 +71,5 @@
 				<parent link="${prefix}_ezgripper_palm_link"/>
 				<child link="${prefix}_ezgripper_finger_${postfix}"/>
-				<origin xyz="0.1056 ${reflectY*0.03} ${reflectZ*0.03}" rpy="${1.5708 * reflectR} 0 3.14159"/>
+				<origin xyz="0.1056 ${reflectY*0.03} 0" rpy="${1.5708 * reflectR} 0 3.14159"/>
 				<axis xyz="0 1 0"/>
 				<limit lower="-.27" upper="1.57075" effort="1" velocity="3.67"/>
@@ -85,5 +79,5 @@
 			</joint>
 	</xacro:macro>
-			<!-- transmissions for Gazebo -->
+	<!-- transmissions for Gazebo -->
 	<xacro:macro name="ezgripper_knuckle_trans" params="prefix postfix">
 		<transmission name="${prefix}_ezgripper_trans_${postfix}">
@@ -99,13 +93,13 @@
 	</xacro:macro>
 	<xacro:macro name="gazebo_knuckle_jsp" params="prefix">
-			<gazebo>
-				<plugin name="joint_state_publisher" filename="libgazebo_ros_joint_state_publisher.so">
-					<jointName>${prefix}_ezgripper_knuckle_1</jointName>
-				</plugin>
-			</gazebo>
+		<gazebo>
+			<plugin name="joint_state_publisher" filename="libgazebo_ros_joint_state_publisher.so">
+				<jointName>${prefix}_ezgripper_knuckle_1</jointName>
+			</plugin>
+		</gazebo>
 	</xacro:macro>
 	<gazebo>
 		<plugin name="gazebo_ros_control" filename="libgazebo_ros_control.so">
-			<robotNamespace>ezgripper_quad</robotNamespace>
+			<robotNamespace>ezgripper_dual_gen1</robotNamespace>
 			<legacyModeNS>true</legacyModeNS>
 		</plugin>
@@ -115,12 +109,4 @@
 			<mimicJoint>left_ezgripper_knuckle_2</mimicJoint>
 		</plugin>
-		<plugin filename="libroboticsgroup_upatras_gazebo_mimic_joint_plugin.so" name="mimicker">
-			<joint>left_ezgripper_knuckle_1</joint>
-			<mimicJoint>left_ezgripper_knuckle_3</mimicJoint>
-		</plugin>
-		<plugin filename="libroboticsgroup_upatras_gazebo_mimic_joint_plugin.so" name="mimicker">
-			<joint>left_ezgripper_knuckle_1</joint>
-			<mimicJoint>left_ezgripper_knuckle_4</mimicJoint>
-		</plugin>
 	</gazebo>
 </robot>

File: ezgripper_description/urdf/dual_gen1/ezgripper_dual_gen1_standalone.urdf.xacro (robot description, xacro)
@@ -4,6 +4,6 @@
 	<xacro:property name="ezgripper_offset_y" value="0.0"/>
 	<xacro:property name="ezgripper_offset_z" value="0.3"/>
-	<xacro:include filename="$(find ezgripper_driver)/urdf/materials.urdf.xacro"/>
-	<xacro:include filename="$(find ezgripper_driver)/urdf/dual_gen1/ezgripper_dual_gen1.urdf.xacro"/>
+	<xacro:include filename="$(find ezgripper_description)/urdf/materials.urdf.xacro"/>
+	<xacro:include filename="$(find ezgripper_description)/urdf/dual_gen1/ezgripper_dual_gen1.urdf.xacro"/>
 	<!-- Add the gripper -->
 	<xacro:ezgripper_dual_gen1 prefix="left" parent_link="base_link">

File: ezgripper_description/urdf/dual_gen2/ezgripper_dual_gen2_articulated.urdf.xacro (robot description, xacro)
@@ -7,5 +7,5 @@
 					<origin xyz="0 0 0" rpy="0 0 0"/>
 					<geometry>
-						<mesh filename="package://ezgripper_driver/meshes/dual_gen2/SAKE_Palm_Dual_Gen2.stl"/>
+						<mesh filename="package://ezgripper_description/meshes/dual_gen2/SAKE_Palm_Dual_Gen2.stl"/>
 					</geometry>
 					<material name="blue"/>
@@ -14,5 +14,5 @@
 					<origin xyz="0 0 0" rpy="0 0 0"/>
 					<geometry>
-						<mesh filename="package://ezgripper_driver/meshes/dual_gen2/SAKE_Palm_Dual_Gen2.stl"/>
+						<mesh filename="package://ezgripper_description/meshes/dual_gen2/SAKE_Palm_Dual_Gen2.stl"/>
 					</geometry>
 				</collision>
@@ -50,5 +50,5 @@
 					<origin xyz="0 0 0" rpy="0 0 0"/>
 					<geometry>
-						<mesh filename="package://ezgripper_driver/meshes/dual_gen2/SAKE_Finger_L1_Gen2.stl"/>
+						<mesh filename="package://ezgripper_description/meshes/dual_gen2/SAKE_Finger_L1_Gen2.stl"/>
 					</geometry>
 					<material name="grey"/>
@@ -57,5 +57,5 @@
 					<origin xyz="0 0 0" rpy="0 0 0"/>
 					<geometry>
-						<mesh filename="package://ezgripper_driver/meshes/dual_gen2/SAKE_Finger_L1_Gen2.stl"/>
+						<mesh filename="package://ezgripper_description/meshes/dual_gen2/SAKE_Finger_L1_Gen2.stl"/>
 					</geometry>
 				</collision>
@@ -74,5 +74,5 @@
 					<origin xyz="0 0 0" rpy="0 0 0"/>
 					<geometry>
-						<mesh filename="package://ezgripper_driver/meshes/dual_gen2/SAKE_Finger_L2_Gen2.stl"/>
+						<mesh filename="package://ezgripper_description/meshes/dual_gen2/SAKE_Finger_L2_Gen2.stl"/>
 					</geometry>
 					<material name="grey"/>
@@ -81,5 +81,5 @@
 					<origin xyz="0 0 0" rpy="0 0 0"/>
 					<geometry>
-						<mesh filename="package://ezgripper_driver/meshes/dual_gen2/SAKE_Finger_L2_Gen2.stl"/>
+						<mesh filename="package://ezgripper_description/meshes/dual_gen2/SAKE_Finger_L2_Gen2.stl"/>
 					</geometry>
 				</collision>

File: ezgripper_description/urdf/dual_gen2/ezgripper_dual_gen2_standalone.urdf.xacro (robot description, xacro)
@@ -4,6 +4,6 @@
 	<xacro:property name="ezgripper_offset_y" value="0.0"/>
 	<xacro:property name="ezgripper_offset_z" value="0.3"/>
-	<xacro:include filename="$(find ezgripper_driver)/urdf/materials.urdf.xacro"/>
-	<xacro:include filename="$(find ezgripper_driver)/urdf/dual_gen2/ezgripper_dual_gen2_articulated.urdf.xacro"/>
+	<xacro:include filename="$(find ezgripper_description)/urdf/materials.urdf.xacro"/>
+	<xacro:include filename="$(find ezgripper_description)/urdf/dual_gen2/ezgripper_dual_gen2_articulated.urdf.xacro"/>
 	<!-- Add the gripper -->
 	<xacro:ezgripper_dual_gen2 prefix="left" parent_link="base_link">

File: ezgripper_description/urdf/quad/ezgripper_quad.urdf.xacro (robot description, xacro)
@@ -1,5 +1,5 @@
 <?xml version="1.0" encoding="UTF-8"?>
-<robot name="ezgripper_dual_gen1" xmlns:xacro="http://ros.org/wiki/xacro">
-	<xacro:macro name="ezgripper_dual_gen1" params="prefix parent_link *origin">
+<robot name="ezgripper_quad" xmlns:xacro="http://ros.org/wiki/xacro">
+	<xacro:macro name="ezgripper_quad" params="prefix parent_link *origin">
 			<!-- links -->
 			<link name="${prefix}_ezgripper_palm_link">
@@ -7,5 +7,5 @@
 					<origin xyz="0 0 0" rpy="0 0 0"/>
 					<geometry>
-						<mesh filename="package://ezgripper_driver/meshes/dual_gen1/SAKE_Palm_Dual.stl"/>
+						<mesh filename="package://ezgripper_description/meshes/quad/SAKE_Palm_Quad.stl"/>
 					</geometry>
 					<material name="blue"/>
@@ -14,5 +14,5 @@
 					<origin xyz="0 0 0" rpy="0 0 0"/>
 					<geometry>
-						<mesh filename="package://ezgripper_driver/meshes/dual_gen1/SAKE_Palm_Dual.stl"/>
+						<mesh filename="package://ezgripper_description/meshes/quad/SAKE_Palm_Quad.stl"/>
 					</geometry>
 				</collision>
@@ -32,12 +32,18 @@
 					<limit effort="0" lower="-1.57075" upper="0.25" velocity="3.67"/>
 			</joint>
-			<xacro:ezgripper_finger prefix="${prefix}" postfix="1" reflect="1" />
-			<xacro:ezgripper_finger prefix="${prefix}" postfix="2" reflect="1" />
-			<!-- Mimic Test has to set be false for the first joint -->
+			<xacro:ezgripper_finger prefix="${prefix}" postfix="1" reflect="1"/>
+			<xacro:ezgripper_finger prefix="${prefix}" postfix="2" reflect="1"/>
+			<xacro:ezgripper_finger prefix="${prefix}" postfix="3" reflect="1"/>
+			<xacro:ezgripper_finger prefix="${prefix}" postfix="4" reflect="1"/>
+			<!-- Mimic Test has to be set false for the first joint -->
 			<xacro:ezgripper_knuckle prefix="${prefix}" postfix="1" reflectY="1" reflectZ="1" reflectR="1" mimic_test="false"/>
 			<xacro:ezgripper_knuckle prefix="${prefix}" postfix="2" reflectY="-1" reflectZ="1" reflectR="-1" mimic_test="true"/>
+			<xacro:ezgripper_knuckle prefix="${prefix}" postfix="3" reflectY="1" reflectZ="-1" reflectR="1" mimic_test="true"/>
+			<xacro:ezgripper_knuckle prefix="${prefix}" postfix="4" reflectY="-1" reflectZ="-1" reflectR="-1" mimic_test="true"/>
 			<!-- Transmission needs to be removed when mimicked -->
 			<xacro:ezgripper_knuckle_trans prefix="${prefix}" postfix="1"/>
-			<!-- <xacro:ezgripper_knuckle_trans prefix="${prefix}" postfix="2"/> -->
+			<!-- <xacro:ezgripper_knuckle_trans prefix="${prefix}" postfix="2"/>
+			<xacro:ezgripper_knuckle_trans prefix="${prefix}" postfix="3"/>
+			<xacro:ezgripper_knuckle_trans prefix="${prefix}" postfix="4"/> -->
 			<xacro:gazebo_knuckle_jsp prefix="${prefix}" />
 	</xacro:macro>
@@ -47,5 +53,5 @@
 					<origin xyz="0 0 0" rpy="0 0 0"/>
 					<geometry>
-						<mesh filename="package://ezgripper_driver/meshes/dual_gen1/SAKE_Finger.stl"/>
+						<mesh filename="package://ezgripper_description/meshes/quad/SAKE_Finger.stl"/>
 					</geometry>
 					<material name="grey"/>
@@ -54,10 +60,10 @@
 					<origin xyz="0 0 0" rpy="0 0 0"/>
 					<geometry>
-						<mesh filename="package://ezgripper_driver/meshes/dual_gen1/SAKE_Finger.stl"/>
+						<mesh filename="package://ezgripper_description/meshes/quad/SAKE_Finger.stl"/>
 					</geometry>
 				</collision>
 				<inertial>
 					<mass value=".025"/>
-					<inertia ixx="0.01" ixy="0.0" ixz="0.0" iyy="0.01" iyz="0.0" izz="0.01"/>
+					<inertia ixx="0.01" ixy="0.0" ixz="0.0" iyy=".01" iyz="0.0" izz="0.01"/>
 				</inertial>
 			</link>
@@ -71,5 +77,5 @@
 				<parent link="${prefix}_ezgripper_palm_link"/>
 				<child link="${prefix}_ezgripper_finger_${postfix}"/>
-				<origin xyz="0.1056 ${reflectY*0.03} 0" rpy="${1.5708 * reflectR} 0 3.14159"/>
+				<origin xyz="0.1056 ${reflectY*0.03} ${reflectZ*0.03}" rpy="${1.5708 * reflectR} 0 3.14159"/>
 				<axis xyz="0 1 0"/>
 				<limit lower="-.27" upper="1.57075" effort="1" velocity="3.67"/>
@@ -79,5 +85,5 @@
 			</joint>
 	</xacro:macro>
-	<!-- transmissions for Gazebo -->
+			<!-- transmissions for Gazebo -->
 	<xacro:macro name="ezgripper_knuckle_trans" params="prefix postfix">
 		<transmission name="${prefix}_ezgripper_trans_${postfix}">
@@ -93,13 +99,13 @@
 	</xacro:macro>
 	<xacro:macro name="gazebo_knuckle_jsp" params="prefix">
-		<gazebo>
-			<plugin name="joint_state_publisher" filename="libgazebo_ros_joint_state_publisher.so">
-				<jointName>${prefix}_ezgripper_knuckle_1</jointName>
-			</plugin>
-		</gazebo>
+			<gazebo>
+				<plugin name="joint_state_publisher" filename="libgazebo_ros_joint_state_publisher.so">
+					<jointName>${prefix}_ezgripper_knuckle_1</jointName>
+				</plugin>
+			</gazebo>
 	</xacro:macro>
 	<gazebo>
 		<plugin name="gazebo_ros_control" filename="libgazebo_ros_control.so">
-			<robotNamespace>ezgripper_dual_gen1</robotNamespace>
+			<robotNamespace>ezgripper_quad</robotNamespace>
 			<legacyModeNS>true</legacyModeNS>
 		</plugin>
@@ -109,4 +115,12 @@
 			<mimicJoint>left_ezgripper_knuckle_2</mimicJoint>
 		</plugin>
+		<plugin filename="libroboticsgroup_upatras_gazebo_mimic_joint_plugin.so" name="mimicker">
+			<joint>left_ezgripper_knuckle_1</joint>
+			<mimicJoint>left_ezgripper_knuckle_3</mimicJoint>
+		</plugin>
+		<plugin filename="libroboticsgroup_upatras_gazebo_mimic_joint_plugin.so" name="mimicker">
+			<joint>left_ezgripper_knuckle_1</joint>
+			<mimicJoint>left_ezgripper_knuckle_4</mimicJoint>
+		</plugin>
 	</gazebo>
 </robot>

File: ezgripper_description/urdf/quad/ezgripper_quad_standalone.urdf.xacro (robot description, xacro)
@@ -4,6 +4,6 @@
 	<xacro:property name="ezgripper_offset_y" value="0.0"/>
 	<xacro:property name="ezgripper_offset_z" value="0.3"/>
-	<xacro:include filename="$(find ezgripper_driver)/urdf/materials.urdf.xacro"/>
-	<xacro:include filename="$(find ezgripper_driver)/urdf/quad/ezgripper_quad.urdf.xacro"/>
+	<xacro:include filename="$(find ezgripper_description)/urdf/materials.urdf.xacro"/>
+	<xacro:include filename="$(find ezgripper_description)/urdf/quad/ezgripper_quad.urdf.xacro"/>
 	<!-- Add the gripper -->
 	<xacro:ezgripper_quad prefix="left" parent_link="base_link">
