Commit message: added single_mount and triple_mount

File: ezgripper_description/urdf/dual_gen1/ezgripper_dual_gen1.urdf.xacro (robot description, xacro)
@@ -2,80 +2,80 @@
 <robot name="ezgripper_dual_gen1" xmlns:xacro="http://ros.org/wiki/xacro">
 	<xacro:macro name="ezgripper_dual_gen1" params="prefix parent_link *origin">
-			<!-- links -->
-			<link name="${prefix}_ezgripper_palm_link">
-				<visual>
-					<origin xyz="0 0 0" rpy="0 0 0"/>
-					<geometry>
-						<mesh filename="package://ezgripper_description/meshes/dual_gen1/SAKE_Palm_Dual.stl"/>
-					</geometry>
-					<material name="blue"/>
-				</visual>
-				<collision>
-					<origin xyz="0 0 0" rpy="0 0 0"/>
-					<geometry>
-						<mesh filename="package://ezgripper_description/meshes/dual_gen1/SAKE_Palm_Dual.stl"/>
-					</geometry>
-				</collision>
+		<!-- links -->
+		<link name="${prefix}_ezgripper_palm_link">
+			<visual>
+				<origin xyz="0 0 0" rpy="0 0 0"/>
+				<geometry>
+					<mesh filename="package://ezgripper_description/meshes/dual_gen1/SAKE_Palm_Dual.stl"/>
+				</geometry>
+				<material name="blue"/>
+			</visual>
+			<collision>
+				<origin xyz="0 0 0" rpy="0 0 0"/>
+				<geometry>
+					<mesh filename="package://ezgripper_description/meshes/dual_gen1/SAKE_Palm_Dual.stl"/>
+				</geometry>
+			</collision>
 			<inertial>
 				<mass value=".3"/>
 				<inertia ixx="0.01" ixy="0.0" ixz="0.0" iyy="0.01" iyz="0.0" izz="0.01"/>
 			</inertial>
-			</link>
-			<gazebo reference="${prefix}_ezgripper_palm_link">
-				<material>Gazebo/Blue</material>
+		</link>
+		<gazebo reference="${prefix}_ezgripper_palm_link">
+			<material>Gazebo/Blue</material>
 		</gazebo>
-			<joint name="${prefix}_ezgripper_connect" type="fixed">
-					<xacro:insert_block name="origin" />
-					<parent link="${parent_link}"/>
-					<child link="${prefix}_ezgripper_palm_link"/>
-					<axis xyz="0 0 0"/>
-					<limit effort="0" lower="-1.57075" upper="0.25" velocity="3.67"/>
-			</joint>
-			<xacro:ezgripper_finger prefix="${prefix}" postfix="1" reflect="1" />
-			<xacro:ezgripper_finger prefix="${prefix}" postfix="2" reflect="1" />
-			<!-- Mimic Test has to set be false for the first joint -->
-			<xacro:ezgripper_knuckle prefix="${prefix}" postfix="1" reflectY="1" reflectZ="1" reflectR="1" mimic_test="false"/>
-			<xacro:ezgripper_knuckle prefix="${prefix}" postfix="2" reflectY="-1" reflectZ="1" reflectR="-1" mimic_test="true"/>
-			<!-- Transmission needs to be removed when mimicked -->
-			<xacro:ezgripper_knuckle_trans prefix="${prefix}" postfix="1"/>
-			<!-- <xacro:ezgripper_knuckle_trans prefix="${prefix}" postfix="2"/> -->
-			<xacro:gazebo_knuckle_jsp prefix="${prefix}" />
+		<joint name="${prefix}_ezgripper_connect" type="fixed">
+				<xacro:insert_block name="origin" />
+				<parent link="${parent_link}"/>
+				<child link="${prefix}_ezgripper_palm_link"/>
+				<axis xyz="0 0 0"/>
+				<limit effort="0" lower="-1.57075" upper="0.25" velocity="3.67"/>
+		</joint>
+		<xacro:ezgripper_finger prefix="${prefix}" postfix="1" reflect="1" />
+		<xacro:ezgripper_finger prefix="${prefix}" postfix="2" reflect="1" />
+		<!-- Mimic Test has to set be false for the first joint -->
+		<xacro:ezgripper_knuckle prefix="${prefix}" postfix="1" reflectY="1" reflectZ="1" reflectR="1" mimic_test="false"/>
+		<xacro:ezgripper_knuckle prefix="${prefix}" postfix="2" reflectY="-1" reflectZ="1" reflectR="-1" mimic_test="true"/>
+		<!-- Transmission needs to be removed when mimicked -->
+		<xacro:ezgripper_knuckle_trans prefix="${prefix}" postfix="1"/>
+		<!-- <xacro:ezgripper_knuckle_trans prefix="${prefix}" postfix="2"/> -->
+		<xacro:gazebo_knuckle_jsp prefix="${prefix}" />
 	</xacro:macro>
 	<xacro:macro name="ezgripper_finger" params="prefix postfix reflect">
-			<link name="${prefix}_ezgripper_finger_${postfix}">
-				<visual>
-					<origin xyz="0 0 0" rpy="0 0 0"/>
-					<geometry>
-						<mesh filename="package://ezgripper_description/meshes/dual_gen1/SAKE_Finger.stl"/>
-					</geometry>
-					<material name="grey"/>
-				</visual>
-				<collision>
-					<origin xyz="0 0 0" rpy="0 0 0"/>
-					<geometry>
-						<mesh filename="package://ezgripper_description/meshes/dual_gen1/SAKE_Finger.stl"/>
-					</geometry>
-				</collision>
-				<inertial>
-					<mass value=".025"/>
-					<inertia ixx="0.01" ixy="0.0" ixz="0.0" iyy="0.01" iyz="0.0" izz="0.01"/>
-				</inertial>
-			</link>
-			<gazebo reference="${prefix}_ezgripper_finger_${postfix}">
-				<material>Gazebo/Grey</material>
+		<link name="${prefix}_ezgripper_finger_${postfix}">
+			<visual>
+				<origin xyz="0 0 0" rpy="0 0 0"/>
+				<geometry>
+					<mesh filename="package://ezgripper_description/meshes/dual_gen1/SAKE_Finger.stl"/>
+				</geometry>
+				<material name="grey"/>
+			</visual>
+			<collision>
+				<origin xyz="0 0 0" rpy="0 0 0"/>
+				<geometry>
+					<mesh filename="package://ezgripper_description/meshes/dual_gen1/SAKE_Finger.stl"/>
+				</geometry>
+			</collision>
+			<inertial>
+				<mass value=".025"/>
+				<inertia ixx="0.01" ixy="0.0" ixz="0.0" iyy="0.01" iyz="0.0" izz="0.01"/>
+			</inertial>
+		</link>
+		<gazebo reference="${prefix}_ezgripper_finger_${postfix}">
+			<material>Gazebo/Grey</material>
 		</gazebo>
 	</xacro:macro>
 	<!-- joints -->
 	<xacro:macro name="ezgripper_knuckle" params="prefix postfix reflectY reflectZ reflectR mimic_test">
-			<joint name="${prefix}_ezgripper_knuckle_${postfix}" type="revolute">
-				<parent link="${prefix}_ezgripper_palm_link"/>
-				<child link="${prefix}_ezgripper_finger_${postfix}"/>
-				<origin xyz="0.1056 ${reflectY*0.03} 0" rpy="${1.5708 * reflectR} 0 3.14159"/>
-				<axis xyz="0 1 0"/>
-				<limit lower="-.27" upper="1.57075" effort="1" velocity="3.67"/>
-				<xacro:if value="${mimic_test}">
-						<mimic joint="${prefix}_ezgripper_knuckle_1"/>
-				</xacro:if>
-			</joint>
+		<joint name="${prefix}_ezgripper_knuckle_${postfix}" type="revolute">
+			<parent link="${prefix}_ezgripper_palm_link"/>
+			<child link="${prefix}_ezgripper_finger_${postfix}"/>
+			<origin xyz="0.1056 ${reflectY*0.03} 0" rpy="${1.5708 * reflectR} 0 3.14159"/>
+			<axis xyz="0 1 0"/>
+			<limit lower="-.27" upper="1.57075" effort="1" velocity="3.67"/>
+			<xacro:if value="${mimic_test}">
+					<mimic joint="${prefix}_ezgripper_knuckle_1"/>
+			</xacro:if>
+		</joint>
 	</xacro:macro>
 	<!-- transmissions for Gazebo -->

File: ezgripper_description/urdf/dual_gen1/ezgripper_dual_gen1_standalone.urdf.xacro (robot description, xacro)
@@ -17,16 +17,16 @@
 	<link name="base_link">
 		<visual>
-				<geometry>
-						<cylinder length="0.42" radius="0.02"/>
-					</geometry>
-					<origin rpy="0 0 0" xyz="0 0 0.21"/>
-					<material name="black"/>
-			</visual>
-			<collision>
-				<geometry>
-						<cylinder length="0.42" radius="0.02"/>
-				</geometry>
-				<origin rpy="0 0 0" xyz="0 0 0.21"/>
-			</collision>
+			<geometry>
+				<cylinder length="0.42" radius="0.02"/>
+			</geometry>
+			<origin rpy="0 0 0" xyz="0 0 0.21"/>
+			<material name="black"/>
+		</visual>
+		<collision>
+			<geometry>
+				<cylinder length="0.42" radius="0.02"/>
+			</geometry>
+			<origin rpy="0 0 0" xyz="0 0 0.21"/>
+		</collision>
 	</link>
 	<gazebo reference="base_link">

File: ezgripper_description/urdf/dual_gen2/ezgripper_dual_gen2_articulated.urdf.xacro (robot description, xacro)
@@ -3,114 +3,114 @@
 	<xacro:macro name="ezgripper_dual_gen2" params="prefix parent_link *origin">
 			<!-- links -->
-			<link name="${prefix}_ezgripper_palm_link">
-				<visual>
-					<origin xyz="0 0 0" rpy="0 0 0"/>
-					<geometry>
-						<mesh filename="package://ezgripper_description/meshes/dual_gen2/SAKE_Palm_Dual_Gen2.stl"/>
-					</geometry>
-					<material name="blue"/>
-				</visual>
-				<collision>
-					<origin xyz="0 0 0" rpy="0 0 0"/>
-					<geometry>
-						<mesh filename="package://ezgripper_description/meshes/dual_gen2/SAKE_Palm_Dual_Gen2.stl"/>
-					</geometry>
-				</collision>
-				<inertial>
-					<mass value=".3"/>
-					<inertia ixx="0.01" ixy="0.0" ixz="0.0" iyy="0.01" iyz="0.0" izz="0.01"/>
-				</inertial>
-			</link>
-			<gazebo reference="${prefix}_ezgripper_palm_link">
-				<material>Gazebo/Blue</material>
+		<link name="${prefix}_ezgripper_palm_link">
+			<visual>
+				<origin xyz="0 0 0" rpy="0 0 0"/>
+				<geometry>
+					<mesh filename="package://ezgripper_description/meshes/dual_gen2/SAKE_Palm_Dual_Gen2.stl"/>
+				</geometry>
+				<material name="blue"/>
+			</visual>
+			<collision>
+				<origin xyz="0 0 0" rpy="0 0 0"/>
+				<geometry>
+					<mesh filename="package://ezgripper_description/meshes/dual_gen2/SAKE_Palm_Dual_Gen2.stl"/>
+				</geometry>
+			</collision>
+			<inertial>
+				<mass value=".3"/>
+				<inertia ixx="0.01" ixy="0.0" ixz="0.0" iyy="0.01" iyz="0.0" izz="0.01"/>
+			</inertial>
+		</link>
+		<gazebo reference="${prefix}_ezgripper_palm_link">
+			<material>Gazebo/Blue</material>
 		</gazebo>
-			<joint name="${prefix}_ezgripper_connect" type="fixed">
-					<xacro:insert_block name="origin" />
-					<parent link="${parent_link}"/>
-					<child link="${prefix}_ezgripper_palm_link"/>
-					<axis xyz="0 0 0"/>
-			</joint>
-			<xacro:ezgripper_finger_L1 prefix="${prefix}" postfix="1" reflect="1" />
-			<xacro:ezgripper_finger_L1 prefix="${prefix}" postfix="2" reflect="1" />
-			<xacro:ezgripper_finger_L2 prefix="${prefix}" postfix="1" reflect="1" />
-			<xacro:ezgripper_finger_L2 prefix="${prefix}" postfix="2" reflect="1" />
-			<!-- Mimic Test has to be set false for the first joint -->
-			<xacro:ezgripper_knuckle_palm_L1 prefix="${prefix}" postfix="1" reflectY="1" reflectZ="1" reflectR="1" mimic_test="false" />
-			<xacro:ezgripper_knuckle_palm_L1 prefix="${prefix}" postfix="2" reflectY="-1" reflectZ="1" reflectR="-1" mimic_test="true" />
-			<xacro:ezgripper_knuckle_L1_L2 prefix="${prefix}" postfix="1" reflectY="1" reflectZ="1" reflectR="-1" />
-			<xacro:ezgripper_knuckle_L1_L2 prefix="${prefix}" postfix="2" reflectY="-1" reflectZ="1" reflectR="1" />
-			<!-- Transmission needs to be removed when mimicked -->
-			<xacro:ezgripper_knuckle_palm_trans prefix="${prefix}" postfix="L1_1"/>
-			<!-- <xacro:ezgripper_knuckle_palm_trans prefix="${prefix}" postfix="L1_2"/> -->
-			<xacro:gazebo_knuckle_jsp prefix="${prefix}" />
+		<joint name="${prefix}_ezgripper_connect" type="fixed">
+				<xacro:insert_block name="origin" />
+				<parent link="${parent_link}"/>
+				<child link="${prefix}_ezgripper_palm_link"/>
+				<axis xyz="0 0 0"/>
+		</joint>
+		<xacro:ezgripper_finger_L1 prefix="${prefix}" postfix="1" reflect="1" />
+		<xacro:ezgripper_finger_L1 prefix="${prefix}" postfix="2" reflect="1" />
+		<xacro:ezgripper_finger_L2 prefix="${prefix}" postfix="1" reflect="1" />
+		<xacro:ezgripper_finger_L2 prefix="${prefix}" postfix="2" reflect="1" />
+		<!-- Mimic Test has to be set false for the first joint -->
+		<xacro:ezgripper_knuckle_palm_L1 prefix="${prefix}" postfix="1" reflectY="1" reflectZ="1" reflectR="1" mimic_test="false" />
+		<xacro:ezgripper_knuckle_palm_L1 prefix="${prefix}" postfix="2" reflectY="-1" reflectZ="1" reflectR="-1" mimic_test="true" />
+		<xacro:ezgripper_knuckle_L1_L2 prefix="${prefix}" postfix="1" reflectY="1" reflectZ="1" reflectR="-1" />
+		<xacro:ezgripper_knuckle_L1_L2 prefix="${prefix}" postfix="2" reflectY="-1" reflectZ="1" reflectR="1" />
+		<!-- Transmission needs to be removed when mimicked -->
+		<xacro:ezgripper_knuckle_palm_trans prefix="${prefix}" postfix="L1_1"/>
+		<!-- <xacro:ezgripper_knuckle_palm_trans prefix="${prefix}" postfix="L1_2"/> -->
+		<xacro:gazebo_knuckle_jsp prefix="${prefix}" />
 	</xacro:macro>
 	<xacro:macro name="ezgripper_finger_L1" params="prefix postfix reflect">
-			<link name="${prefix}_ezgripper_finger_L1_${postfix}">
-				<visual>
-					<origin xyz="0 0 0" rpy="0 0 0"/>
-					<geometry>
-						<mesh filename="package://ezgripper_description/meshes/dual_gen2/SAKE_Finger_L1_Gen2.stl"/>
-					</geometry>
-					<material name="grey"/>
-				</visual>
-				<collision>
-					<origin xyz="0 0 0" rpy="0 0 0"/>
-					<geometry>
-						<mesh filename="package://ezgripper_description/meshes/dual_gen2/SAKE_Finger_L1_Gen2.stl"/>
-					</geometry>
-				</collision>
-				<inertial>
-					<mass value=".025"/>
-					<inertia ixx="0.01" ixy="0.0" ixz="0.0" iyy="0.01" iyz="0.0" izz="0.01"/>
-				</inertial>
-			</link>
-			<gazebo reference="${prefix}_ezgripper_finger_L1_${postfix}">
-				<material>Gazebo/Grey</material>
+		<link name="${prefix}_ezgripper_finger_L1_${postfix}">
+			<visual>
+				<origin xyz="0 0 0" rpy="0 0 0"/>
+				<geometry>
+					<mesh filename="package://ezgripper_description/meshes/dual_gen2/SAKE_Finger_L1_Gen2.stl"/>
+				</geometry>
+				<material name="grey"/>
+			</visual>
+			<collision>
+				<origin xyz="0 0 0" rpy="0 0 0"/>
+				<geometry>
+					<mesh filename="package://ezgripper_description/meshes/dual_gen2/SAKE_Finger_L1_Gen2.stl"/>
+				</geometry>
+			</collision>
+			<inertial>
+				<mass value=".025"/>
+				<inertia ixx="0.01" ixy="0.0" ixz="0.0" iyy="0.01" iyz="0.0" izz="0.01"/>
+			</inertial>
+		</link>
+		<gazebo reference="${prefix}_ezgripper_finger_L1_${postfix}">
+			<material>Gazebo/Grey</material>
 		</gazebo>
 	</xacro:macro>
 	<xacro:macro name="ezgripper_finger_L2" params="prefix postfix reflect">
-			<link name="${prefix}_ezgripper_finger_L2_${postfix}">
-				<visual>
-					<origin xyz="0 0 0" rpy="0 0 0"/>
-					<geometry>
-						<mesh filename="package://ezgripper_description/meshes/dual_gen2/SAKE_Finger_L2_Gen2.stl"/>
-					</geometry>
-					<material name="grey"/>
-				</visual>
-				<collision>
-					<origin xyz="0 0 0" rpy="0 0 0"/>
-					<geometry>
-						<mesh filename="package://ezgripper_description/meshes/dual_gen2/SAKE_Finger_L2_Gen2.stl"/>
-					</geometry>
-				</collision>
-				<inertial>
-					<mass value=".025"/>
-					<inertia ixx="0.01" ixy="0.0" ixz="0.0" iyy="0.01" iyz="0.0" izz="0.01"/>
-				</inertial>
-			</link>
-			<gazebo reference="${prefix}_ezgripper_finger_L2_${postfix}">
-				<material>Gazebo/Grey</material>
+		<link name="${prefix}_ezgripper_finger_L2_${postfix}">
+			<visual>
+				<origin xyz="0 0 0" rpy="0 0 0"/>
+				<geometry>
+					<mesh filename="package://ezgripper_description/meshes/dual_gen2/SAKE_Finger_L2_Gen2.stl"/>
+				</geometry>
+				<material name="grey"/>
+			</visual>
+			<collision>
+				<origin xyz="0 0 0" rpy="0 0 0"/>
+				<geometry>
+					<mesh filename="package://ezgripper_description/meshes/dual_gen2/SAKE_Finger_L2_Gen2.stl"/>
+				</geometry>
+			</collision>
+			<inertial>
+				<mass value=".025"/>
+				<inertia ixx="0.01" ixy="0.0" ixz="0.0" iyy="0.01" iyz="0.0" izz="0.01"/>
+			</inertial>
+		</link>
+		<gazebo reference="${prefix}_ezgripper_finger_L2_${postfix}">
+			<material>Gazebo/Grey</material>
 		</gazebo>
 	</xacro:macro>
   <!-- Joints -->
 	<xacro:macro name="ezgripper_knuckle_palm_L1" params="prefix postfix reflectY reflectZ reflectR mimic_test">
-			<joint name="${prefix}_ezgripper_knuckle_palm_L1_${postfix}" type="revolute">
-				<parent link="${prefix}_ezgripper_palm_link"/>
-				<child link="${prefix}_ezgripper_finger_L1_${postfix}"/>
-				<origin xyz="0.072569 ${reflectY*0.03} 0" rpy="${-1.5708 * reflectR} 0 ${1.57075 * reflectR}"/>
-				<axis xyz="0 1 0"/>
-				<limit lower="0" upper="1.94" effort="1.0" velocity="3.67"/>
-				<xacro:if value="${mimic_test}">
-						<mimic joint="${prefix}_ezgripper_knuckle_palm_L1_1"/>
-				</xacro:if>
-			</joint>
+		<joint name="${prefix}_ezgripper_knuckle_palm_L1_${postfix}" type="revolute">
+			<parent link="${prefix}_ezgripper_palm_link"/>
+			<child link="${prefix}_ezgripper_finger_L1_${postfix}"/>
+			<origin xyz="0.072569 ${reflectY*0.03} 0" rpy="${-1.5708 * reflectR} 0 ${1.57075 * reflectR}"/>
+			<axis xyz="0 1 0"/>
+			<limit lower="0" upper="1.94" effort="1.0" velocity="3.67"/>
+			<xacro:if value="${mimic_test}">
+					<mimic joint="${prefix}_ezgripper_knuckle_palm_L1_1"/>
+			</xacro:if>
+		</joint>
 	</xacro:macro>
 	<xacro:macro name="ezgripper_knuckle_L1_L2" params="prefix postfix reflectY reflectZ reflectR">
-			<joint name="${prefix}_ezgripper_knuckle_L1_L2_${postfix}" type="fixed">
-				<parent link="${prefix}_ezgripper_finger_L1_${postfix}"/>
-				<child link="${prefix}_ezgripper_finger_L2_${postfix}"/>
-				<origin xyz="0.052 0 0" rpy="0 0 0"/>
-				<axis xyz="0 1 0"/>
-			</joint>
+		<joint name="${prefix}_ezgripper_knuckle_L1_L2_${postfix}" type="fixed">
+			<parent link="${prefix}_ezgripper_finger_L1_${postfix}"/>
+			<child link="${prefix}_ezgripper_finger_L2_${postfix}"/>
+			<origin xyz="0.052 0 0" rpy="0 0 0"/>
+			<axis xyz="0 1 0"/>
+		</joint>
 	</xacro:macro>
   <!-- Transmissions for Gazebo -->

File: ezgripper_description/urdf/dual_gen2/ezgripper_dual_gen2_standalone.urdf.xacro (robot description, xacro)
@@ -17,16 +17,16 @@
 	<link name="base_link">
 		<visual>
-				<geometry>
-						<cylinder length="0.42" radius="0.02"/>
-					</geometry>
-					<origin rpy="0 0 0" xyz="0 0 0.21"/>
-					<material name="black"/>
-			</visual>
-			<collision>
-				<geometry>
-						<cylinder length="0.42" radius="0.02"/>
-				</geometry>
-				<origin rpy="0 0 0" xyz="0 0 0.21"/>
-			</collision>
+			<geometry>
+				<cylinder length="0.42" radius="0.02"/>
+			</geometry>
+			<origin rpy="0 0 0" xyz="0 0 0.21"/>
+			<material name="black"/>
+		</visual>
+		<collision>
+			<geometry>
+					<cylinder length="0.42" radius="0.02"/>
+			</geometry>
+			<origin rpy="0 0 0" xyz="0 0 0.21"/>
+		</collision>
 	</link>
 	<gazebo reference="base_link">
