Commit message: Fixed bottleneck move_group launch by subsampling meshes, added moveit_configs for newer modules

File: ezgripper_description/urdf/dual_gen2/ezgripper_dual_gen2_standalone.urdf.xacro (robot description, xacro)
@@ -5,5 +5,5 @@
 	<xacro:property name="ezgripper_offset_z" value="0.3"/>
 	<xacro:include filename="$(find ezgripper_description)/urdf/materials.urdf.xacro"/>
-	<xacro:include filename="$(find ezgripper_description)/urdf/dual_gen2/ezgripper_dual_gen2_articulated.urdf.xacro"/>
+	<xacro:include filename="$(find ezgripper_description)/urdf/dual_gen2/ezgripper_dual_gen2.urdf.xacro"/>
 	<!-- Add the gripper -->
 	<xacro:ezgripper_dual_gen2 prefix="left" parent_link="base_link">

File: ezgripper_description/urdf/dual_gen2_triple_mount/ezgripper_dual_gen2_triple_mount.urdf.xacro (robot description, xacro)
@@ -7,5 +7,5 @@
 				<origin xyz="0 0 0" rpy="0 0 0"/>
 				<geometry>
-					<mesh filename="package://ezgripper_description/meshes/dual_gen2_triple_mount//SAKE_Triple_Mount.stl"/>
+					<mesh filename="package://ezgripper_description/meshes/dual_gen2_triple_mount/SAKE_Triple_Mount.stl"/>
 				</geometry>
 				<material name="blue"/>
@@ -14,5 +14,5 @@
 				<origin xyz="0 0 0" rpy="0 0 0"/>
 				<geometry>
-					<mesh filename="package://ezgripper_description/meshes/dual_gen2_triple_mount//SAKE_Triple_Mount.stl"/>
+					<mesh filename="package://ezgripper_description/meshes/dual_gen2_triple_mount/SAKE_Triple_Mount.stl"/>
 				</geometry>
 			</collision>
@@ -45,5 +45,5 @@
 				<origin xyz="0.0 0 0" rpy="0 0 0"/>
 				<geometry>
-					<mesh filename="package://ezgripper_description/meshes/dual_gen2_triple_mount//SAKE_Palm_IM.stl"/>
+					<mesh filename="package://ezgripper_description/meshes/dual_gen2_triple_mount/SAKE_Palm_IM.stl"/>
 				</geometry>
 				<material name="blue"/>
@@ -52,5 +52,5 @@
 				<origin xyz="0.0 0 0" rpy="0 0 0"/>
 				<geometry>
-					<mesh filename="package://ezgripper_description/meshes/dual_gen2_triple_mount//SAKE_Palm_IM.stl"/>
+					<mesh filename="package://ezgripper_description/meshes/dual_gen2_triple_mount/SAKE_Palm_IM.stl"/>
 				</geometry>
 			</collision>
@@ -94,5 +94,5 @@
 				<origin xyz="0 0 0" rpy="0 0 0"/>
 				<geometry>
-					<mesh filename="package://ezgripper_description/meshes/dual_gen2_triple_mount//SAKE_Finger_L1_IM.stl"/>
+					<mesh filename="package://ezgripper_description/meshes/dual_gen2_triple_mount/SAKE_Finger_L1_IM.stl"/>
 				</geometry>
 				<material name="grey"/>
@@ -101,5 +101,5 @@
 				<origin xyz="0 0 0" rpy="0 0 0"/>
 				<geometry>
-					<mesh filename="package://ezgripper_description/meshes/dual_gen2_triple_mount//SAKE_Finger_L1_IM.stl"/>
+					<mesh filename="package://ezgripper_description/meshes/dual_gen2_triple_mount/SAKE_Finger_L1_IM.stl"/>
 				</geometry>
 			</collision>
@@ -118,5 +118,5 @@
 				<origin xyz="0 0 0" rpy="0 0 0"/>
 				<geometry>
-					<mesh filename="package://ezgripper_description/meshes/dual_gen2_triple_mount//SAKE_Finger_L2_IM.stl"/>
+					<mesh filename="package://ezgripper_description/meshes/dual_gen2_triple_mount/SAKE_Finger_L2_IM.stl"/>
 				</geometry>
 				<material name="grey"/>
@@ -125,5 +125,5 @@
 				<origin xyz="0 0 0" rpy="0 0 0"/>
 				<geometry>
-					<mesh filename="package://ezgripper_description/meshes/dual_gen2_triple_mount//SAKE_Finger_L2_IM.stl"/>
+					<mesh filename="package://ezgripper_description/meshes/dual_gen2_triple_mount/SAKE_Finger_L2_IM.stl"/>
 				</geometry>
 			</collision>
@@ -142,5 +142,5 @@
 				<origin xyz="0 0 0" rpy="0 0 0"/>
 				<geometry>
-					<mesh filename="package://ezgripper_description/meshes/dual_gen2_triple_mount//SAKE_Finger_Pad_IM.stl"/>
+					<mesh filename="package://ezgripper_description/meshes/dual_gen2_triple_mount/SAKE_Finger_Pad_IM.stl"/>
 				</geometry>
 				<material name="grey"/>
@@ -149,5 +149,5 @@
 				<origin xyz="0 0 0" rpy="0 0 0"/>
 				<geometry>
-					<mesh filename="package://ezgripper_description/meshes/dual_gen2_triple_mount//SAKE_Finger_Pad_IM.stl"/>
+					<mesh filename="package://ezgripper_description/meshes/dual_gen2_triple_mount/SAKE_Finger_Pad_IM.stl"/>
 				</geometry>
 			</collision>
