Commit message: separating back collision and visual meshes

File: ezgripper_description/urdf/ezgripper_single_mount.urdf.xacro (robot description, xacro)
@@ -7,5 +7,5 @@
 				<xacro:insert_block name="origin"/>
 				<geometry>
-					<mesh filename="package://ezgripper_description/meshes/SAKE_Single_Mount.stl"/>
+					<mesh filename="package://ezgripper_description/meshes/visual/SAKE_Single_Mount.stl"/>
 				</geometry>
 				<material name="blue"/>
@@ -14,5 +14,5 @@
 				<xacro:insert_block name="origin"/>
 				<geometry>
-					<mesh filename="package://ezgripper_description/meshes/SAKE_Single_Mount.stl"/>
+					<mesh filename="package://ezgripper_description/meshes/collision/SAKE_Single_Mount.stl"/>
 				</geometry>
 			</collision>
@@ -41,5 +41,5 @@
 				<origin xyz="0.0 0 0" rpy="0 0 0"/>
 				<geometry>
-					<mesh filename="package://ezgripper_description/meshes/SAKE_Palm_IM.stl"/>
+					<mesh filename="package://ezgripper_description/meshes/visual/SAKE_Palm_IM.stl"/>
 				</geometry>
 				<material name="blue"/>
@@ -48,5 +48,5 @@
 				<origin xyz="0.0 0 0" rpy="0 0 0"/>
 				<geometry>
-					<mesh filename="package://ezgripper_description/meshes/SAKE_Palm_IM.stl"/>
+					<mesh filename="package://ezgripper_description/meshes/collision/SAKE_Palm_IM.stl"/>
 				</geometry>
 			</collision>
@@ -88,5 +88,5 @@
 				<origin xyz="0 0 0" rpy="0 0 0"/>
 				<geometry>
-					<mesh filename="package://ezgripper_description/meshes/SAKE_Finger_L1_IM.stl"/>
+					<mesh filename="package://ezgripper_description/meshes/visual/SAKE_Finger_L1_IM.stl"/>
 				</geometry>
 				<material name="grey"/>
@@ -95,5 +95,5 @@
 				<origin xyz="0 0 0" rpy="0 0 0"/>
 				<geometry>
-					<mesh filename="package://ezgripper_description/meshes/SAKE_Finger_L1_IM.stl"/>
+					<mesh filename="package://ezgripper_description/meshes/collision/SAKE_Finger_L1_IM.stl"/>
 				</geometry>
 			</collision>
@@ -112,5 +112,5 @@
 				<origin xyz="0 0 0" rpy="0 0 0"/>
 				<geometry>
-					<mesh filename="package://ezgripper_description/meshes/SAKE_Finger_L2_IM.stl"/>
+					<mesh filename="package://ezgripper_description/meshes/visual/SAKE_Finger_L2_IM.stl"/>
 				</geometry>
 				<material name="grey"/>
@@ -119,5 +119,5 @@
 				<origin xyz="0 0 0" rpy="0 0 0"/>
 				<geometry>
-					<mesh filename="package://ezgripper_description/meshes/SAKE_Finger_L2_IM.stl"/>
+					<mesh filename="package://ezgripper_description/meshes/collision/SAKE_Finger_L2_IM.stl"/>
 				</geometry>
 			</collision>
@@ -136,5 +136,5 @@
 				<origin xyz="0 0 0" rpy="0 0 0"/>
 				<geometry>
-					<mesh filename="package://ezgripper_description/meshes/SAKE_Finger_Pad_IM.stl"/>
+					<mesh filename="package://ezgripper_description/meshes/visual/SAKE_Finger_Pad_IM.stl"/>
 				</geometry>
 				<material name="grey"/>
@@ -143,5 +143,5 @@
 				<origin xyz="0 0 0" rpy="0 0 0"/>
 				<geometry>
-					<mesh filename="package://ezgripper_description/meshes/SAKE_Finger_Pad_IM.stl"/>
+					<mesh filename="package://ezgripper_description/meshes/collision/SAKE_Finger_Pad_IM.stl"/>
 				</geometry>
 			</collision>

Commit message: adding prefix to gazebo plugin

File: ezgripper_description/urdf/ezgripper_single_mount.urdf.xacro (robot description, xacro)
@@ -1,5 +1,5 @@
 <?xml version="1.0" encoding="UTF-8"?>
 <robot name="ezgripper_single_mount" xmlns:xacro="http://ros.org/wiki/xacro">
-	<xacro:macro name="ezgripper_single_mount" params="prefix parent_link *origin">
+	<xacro:macro name="ezgripper_single_mount" params="prefix parent_link *origin activate_control:=false">
 		<!-- links -->
 		<link name="${prefix}_ezgripper_mount">
@@ -35,4 +35,12 @@
 			<xacro:insert_block name="origin"/>
 		</xacro:ezgripper_palm>
+		<xacro:if value="${activate_control}">
+			<gazebo>
+				<plugin name="gazebo_ros_control" filename="libgazebo_ros_control.so">
+					<robotNamespace>/ezgripper_single_mount</robotNamespace>
+					<legacyModeNS>true</legacyModeNS>
+				</plugin>
+			</gazebo>
+		</xacro:if>
 	</xacro:macro>
 	<xacro:macro name="ezgripper_palm" params="prefix parent_link *origin">
@@ -82,4 +90,5 @@
 		<!-- <xacro:ezgripper_knuckle_palm_trans prefix="${prefix}" postfix="L1_2"/> -->
 		<xacro:gazebo_knuckle_jsp prefix="${prefix}" />
+		<xacro:gazebo_mimic_plugin prefix="${prefix}" />
 	</xacro:macro>
 	<xacro:macro name="ezgripper_finger_L1" params="prefix postfix reflect">
@@ -201,17 +210,16 @@
 			<plugin name="joint_state_publisher" filename="libgazebo_ros_joint_state_publisher.so">
 				<jointName>${prefix}_ezgripper_knuckle_palm_L1_1</jointName>
+				<updateRate>100.0</updateRate>
 			</plugin>
 		</gazebo>
 	</xacro:macro>
-	<gazebo>
-		<plugin name="gazebo_ros_control" filename="libgazebo_ros_control.so">
-			<robotNamespace>/ezgripper_single_mount</robotNamespace>
-			<legacyModeNS>true</legacyModeNS>
-		</plugin>
-		<!-- Fix mimicking bug -->
-		<plugin filename="libroboticsgroup_upatras_gazebo_mimic_joint_plugin.so" name="mimicker">
-			<joint>left_ezgripper_knuckle_palm_L1_1</joint>
-			<mimicJoint>left_ezgripper_knuckle_palm_L1_2</mimicJoint>
-		</plugin>
-	</gazebo>
+	<xacro:macro name="gazebo_mimic_plugin" params="prefix">
+		<gazebo>
+			<!-- Fix mimicking bug -->
+			<plugin filename="libroboticsgroup_upatras_gazebo_mimic_joint_plugin.so" name="mimicker">
+				<joint>${prefix}_ezgripper_knuckle_palm_L1_1</joint>
+				<mimicJoint>${prefix}_ezgripper_knuckle_palm_L1_2</mimicJoint>
+			</plugin>
+		</gazebo>
+	</xacro:macro>
 </robot>

File: ezgripper_description/urdf/ezgripper_single_standalone.urdf.xacro (robot description, xacro)
@@ -7,5 +7,5 @@
 	<xacro:include filename="$(find ezgripper_description)/urdf/ezgripper_single_mount.urdf.xacro"/>
 	<!-- Add the gripper -->
-	<xacro:ezgripper_single_mount prefix="left" parent_link="base_link">
+	<xacro:ezgripper_single_mount prefix="left" parent_link="base_link" activate_control="true">
 		<origin xyz="${ezgripper_offset_x} ${ezgripper_offset_y} ${ezgripper_offset_z}" rpy="0 0 0"/>
 	</xacro:ezgripper_single_mount>
